File: Schaakbord/Schaakbord.sch (KiCad schematic (older format))
At the start: 48 parts, among them IC1 M24C04-RMN6TP, IC10 AH3572-SA-7, IC11 MAX6955AAX+, IC2 SN74HC165DR, IC3 AH3572-SA-7, IC4 AH3572-SA-7, IC5 AH3572-SA-7, IC6 AH3572-SA-7, IC7 AH3572-SA-7, IC8 AH3572-SA-7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

Commit message: Update
Parts:
- added C10: 100nF, symbol Device:C
- added C8: 12pF, symbol Device:C
- added C9: 47µF, symbol Device:C
- added R13: 110k, symbol Device:R
- C7: value 40pF -> 20pF
Connections:
- net labels added: O0, O1, O11, O12, O13, O14, O15, O16, O17, O18, O2, O3, O4, O5, O6, O7, O8
- wire segments 151 -> 187
Other:
- moved on the sheet: DS1, IC11
Changed lines of the file:
@@
 P 12750 5050
 F 0 "C7" H 12865 5096 50  0000 L CNN
-F 1 "40pF" H 12865 5005 50  0000 L CNN
+F 1 "20pF" H 12865 5005 50  0000 L CNN
 F 2 "" H 12788 4900 50  0001 C CNN
 F 3 "~" H 12750 5050 50  0001 C CNN
@@
 L SamacSys_Parts:MAX6955AAX+ IC11
 U 1 1 603D7BCA
-P 6500 3300
-F 0 "IC11" H 7150 3565 50  0000 C CNN
-F 1 "MAX6955AAX+" H 7150 3474 50  0000 C CNN
-F 2 "SOP80P1030X264-36N" H 7650 3400 50  0001 L CNN
-F 3 "http://datasheets.maximintegrated.com/en/ds/MAX6955.pdf" H 7650 3300 50  0001 L CNN
-F 4 "MAX6955AAX+, LED Display Driver, 16-Digits 128-Segments, 2.7  5.5 V, 36-Pin SSOP" H 7650 3200 50  0001 L CNN "Description"
-F 5 "2.64" H 7650 3100 50  0001 L CNN "Height"
-F 6 "700-MAX6955AAX" H 7650 3000 50  0001 L CNN "Mouser Part Number"
-F 7 "https://www.mouser.co.uk/ProductDetail/Maxim-Integrated/MAX6955AAX%2b/?qs=1THa7WoU59HHiplILEoAzQ%3D%3D" H 7650 2900 50  0001 L CNN "Mouser Price/Stock"
-F 8 "Maxim Integrated" H 7650 2800 50  0001 L CNN "Manufacturer_Name"
-F 9 "MAX6955AAX+" H 7650 2700 50  0001 L CNN "Manufacturer_Part_Number"
-	1    6500 3300
+P 5850 3300
+F 0 "IC11" H 6500 3565 50  0000 C CNN
+F 1 "MAX6955AAX+" H 6500 3474 50  0000 C CNN
+F 2 "SOP80P1030X264-36N" H 7000 3400 50  0001 L CNN
+F 3 "http://datasheets.maximintegrated.com/en/ds/MAX6955.pdf" H 7000 3300 50  0001 L CNN
+F 4 "MAX6955AAX+, LED Display Driver, 16-Digits 128-Segments, 2.7  5.5 V, 36-Pin SSOP" H 7000 3200 50  0001 L CNN "Description"
+F 5 "2.64" H 7000 3100 50  0001 L CNN "Height"
+F 6 "700-MAX6955AAX" H 7000 3000 50  0001 L CNN "Mouser Part Number"
+F 7 "https://www.mouser.co.uk/ProductDetail/Maxim-Integrated/MAX6955AAX%2b/?qs=1THa7WoU59HHiplILEoAzQ%3D%3D" H 7000 2900 50  0001 L CNN "Mouser Price/Stock"
+F 8 "Maxim Integrated" H 7000 2800 50  0001 L CNN "Manufacturer_Name"
+F 9 "MAX6955AAX+" H 7000 2700 50  0001 L CNN "Manufacturer_Part_Number"
+	1    5850 3300
 	1    0    0    -1
 $EndComp
@@
 L SamacSys_Parts:HDSP-B03G DS1
 U 1 1 603F487A
-P 8450 3700
-F 0 "DS1" H 9900 3965 50  0000 C CNN
-F 1 "HDSP-B03G" H 9900 3874 50  0000 C CNN
-F 2 "HDSPB03G" H 11200 3800 50  0001 L CNN
-F 3 "https://docs.broadcom.com/docs/AV01-0698EN" H 11200 3700 50  0001 L CNN
-F 4 "LED Displays & Accessories 88:88 Clock Module 0.56in 4 Digits CC" H 11200 3600 50  0001 L CNN "Description"
-F 5 "8" H 11200 3500 50  0001 L CNN "Height"
-F 6 "630-HDSP-B03G" H 11200 3400 50  0001 L CNN "Mouser Part Number"
-F 7 "https://www.mouser.co.uk/ProductDetail/Broadcom-Avago/HDSP-B03G/?qs=pQfy5%252BKCabJU4dELvEhWiw%3D%3D" H 11200 3300 50  0001 L CNN "Mouser Price/Stock"
-F 8 "Avago Technologies" H 11200 3200 50  0001 L CNN "Manufacturer_Name"
-F 9 "HDSP-B03G" H 11200 3100 50  0001 L CNN "Manufacturer_Part_Number"
-	1    8450 3700
+P 8450 3350
+F 0 "DS1" H 9900 3615 50  0000 C CNN
+F 1 "HDSP-B03G" H 9900 3524 50  0000 C CNN
+F 2 "HDSPB03G" H 11200 3450 50  0001 L CNN
+F 3 "https://docs.broadcom.com/docs/AV01-0698EN" H 11200 3350 50  0001 L CNN
+F 4 "LED Displays & Accessories 88:88 Clock Module 0.56in 4 Digits CC" H 11200 3250 50  0001 L CNN "Description"
+F 5 "8" H 11200 3150 50  0001 L CNN "Height"
+F 6 "630-HDSP-B03G" H 11200 3050 50  0001 L CNN "Mouser Part Number"
+F 7 "https://www.mouser.co.uk/ProductDetail/Broadcom-Avago/HDSP-B03G/?qs=pQfy5%252BKCabJU4dELvEhWiw%3D%3D" H 11200 2950 50  0001 L CNN "Mouser Price/Stock"
+F 8 "Avago Technologies" H 11200 2850 50  0001 L CNN "Manufacturer_Name"
+F 9 "HDSP-B03G" H 11200 2750 50  0001 L CNN "Manufacturer_Part_Number"
+	1    8450 3350
 	1    0    0    -1
 $EndComp
@@
 	1    0    0    -1
 $EndComp
+$Comp
+L Device:R R13
+U 1 1 604802D6
+P 5600 4900
+F 0 "R13" V 5550 5100 50  0000 C CNN
+F 1 "110k" V 5650 5100 50  0000 C CNN
+F 2 "" V 5530 4900 50  0001 C CNN
+F 3 "~" H 5600 4900 50  0001 C CNN
+	1    5600 4900
+	0    1    1    0
+$EndComp
+Wire Wire Line
+	5400 5000 5850 5000
+Wire Wire Line
+	5850 4800 5400 4800
+Wire Wire Line
+	5400 4800 5400 4900
+Wire Wire Line
+	5450 4900 5400 4900
+Wire Wire Line
+	5750 4900 5850 4900
+Connection ~ 5400 4900
+Wire Wire Line
+	5400 4900 5400 5000
+Wire Wire Line
+	14000 5250 14000 5350
+Connection ~ 14000 5250
+Connection ~ 14000 5350
+$Comp
+L Device:C C8
+U 1 1 604B302F
+P 7700 4900
+F 0 "C8" V 7550 4800 50  0000 C CNN
+F 1 "12pF" V 7550 5000 50  0000 C CNN
+F 2 "" H 7738 4750 50  0001 C CNN
+F 3 "~" H 7700 4900 50  0001 C CNN
+	1    7700 4900
+	0    1    1    0
+$EndComp
+Wire Wire Line
+	7150 4800 7500 4800
+Wire Wire Line
+	7500 4800 7500 5000
+Wire Wire Line
+	7500 5000 7450 5000
+Wire Wire Line
+	7150 4900 7550 4900
+$Comp
+L power:GNDD #PWR064
+U 1 1 604EB109
+P 7450 5350
+F 0 "#PWR064" H 7450 5100 50  0001 C CNN
+F 1 "GNDD" H 7454 5195 50  0000 C CNN
+F 2 "" H 7450 5350 50  0001 C CNN
+F 3 "" H 7450 5350 50  0001 C CNN
+	1    7450 5350
+	1    0    0    -1
+$EndComp
+$Comp
+L power:GNDD #PWR063
+U 1 1 604EB686
+P 5400 5000
+F 0 "#PWR063" H 5400 4750 50  0001 C CNN
+F 1 "GNDD" H 5404 4845 50  0000 C CNN
+F 2 "" H 5400 5000 50  0001 C CNN
+F 3 "" H 5400 5000 50  0001 C CNN
+	1    5400 5000
+	1    0    0    -1
+$EndComp
+Connection ~ 5400 5000
+$Comp
+L Device:C C9
+U 1 1 604FBDA1
+P 7250 5150
+F 0 "C9" H 7450 5100 50  0000 C CNN
+F 1 "47µF" H 7450 5200 50  0000 C CNN
+F 2 "" H 7288 5000 50  0001 C CNN
+F 3 "~" H 7250 5150 50  0001 C CNN
+	1    7250 5150
+	-1   0    0    1
+$EndComp
+$Comp
+L Device:C C10
+U 1 1 60504080
+P 7450 5150
+F 0 "C10" H 7650 5200 50  0000 C CNN
+F 1 "100nF" H 7700 5100 50  0000 C CNN
+F 2 "" H 7488 5000 50  0001 C CNN
+F 3 "~" H 7450 5150 50  0001 C CNN
+	1    7450 5150
+	1    0    0    -1
+$EndComp
+Connection ~ 7450 5000
+Connection ~ 7250 5000
+Wire Wire Line
+	7250 5000 7450 5000
+Wire Wire Line
+	7150 5000 7250 5000
+Wire Wire Line
+	7250 5300 7450 5300
+Wire Wire Line
+	7450 5300 7450 5350
+Connection ~ 7450 5300
+Wire Wire Line
+	7450 5300 7850 5300
+Wire Wire Line
+	7850 5300 7850 4900
+Text GLabel 5750 3700 0    50   Input ~ 0
+PB10
+Wire Wire Line
+	5750 3700 5850 3700
+Text GLabel 5750 3600 0    50   Input ~ 0
+PB11
+Wire Wire Line
+	5750 3600 5850 3600
+Text GLabel 7250 4500 2    50   Input ~ 0
+O11
+Wire Wire Line
+	7150 4500 7250 4500
+Text GLabel 7250 4400 2    50   Input ~ 0
+O12
+Text GLabel 7250 4300 2    50   Input ~ 0
+O13
+Text GLabel 7250 4200 2    50   Input ~ 0
+O14
+Text GLabel 7250 4100 2    50   Input ~ 0
+O15
+Text GLabel 7250 4000 2    50   Input ~ 0
+O16
+Text GLabel 7250 3900 2    50   Input ~ 0
+O17
+Text GLabel 7250 3800 2    50   Input ~ 0
+O18
+Wire Wire Line
+	7250 4400 7150 4400
+Wire Wire Line
+	7250 4300 7150 4300
+Wire Wire Line
+	7250 4200 7150 4200
+Wire Wire Line
+	7250 4100 7150 4100
+Wire Wire Line
+	7250 4000 7150 4000
+Wire Wire Line
+	7250 3900 7150 3900
+Wire Wire Line
+	7250 3800 7150 3800
+Text GLabel 5750 4000 0    50   Input ~ 0
+O1
+Wire Wire Line
+	5750 4000 5850 4000
+Text GLabel 5750 4100 0    50   Input ~ 0
+O2
+Text GLabel 5750 4200 0    50   Input ~ 0
+O3
+Text GLabel 5750 4300 0    50   Input ~ 0
+O4
+Text GLabel 5750 4400 0    50   Input ~ 0
+O5
+Text GLabel 5750 4500 0    50   Input ~ 0
+O6
+Text GLabel 5750 4600 0    50   Input ~ 0
+O7
+Text GLabel 5750 4700 0    50   Input ~ 0
+O8
+Wire Wire Line
+	5750 4700 5850 4700
+Wire Wire Line
+	5750 4600 5850 4600
+Wire Wire Line
+	5750 4500 5850 4500
+Wire Wire Line
+	5750 4400 5850 4400
+Wire Wire Line
+	5750 4300 5850 4300
+Wire Wire Line
+	5750 4200 5850 4200
+Wire Wire Line
+	5750 4100 5850 4100
+Text GLabel 5750 3900 0    50   Input ~ 0
+O0
+Wire Wire Line
+	5750 3900 5850 3900
 $EndSCHEMATC

Commit message: Update Schaakbord.sch
Connections:
- net labels removed: O8
- wire segments 187 -> 212
Other:
- moved on the sheet: DS2
Changed lines of the file:
@@
 	7150 7400 7350 7400
-Wire Wire Line
-	7350 7800 7450 7800
 Wire Wire Line
 	7350 7600 7350 7800
@@
 L power:GNDD #PWR031
 U 1 1 6038D2B1
-P 7450 7800
-F 0 "#PWR031" H 7450 7550 50  0001 C CNN
-F 1 "GNDD" H 7454 7645 50  0000 C CNN
-F 2 "" H 7450 7800 50  0001 C CNN
-F 3 "" H 7450 7800 50  0001 C CNN
-	1    7450 7800
-	1    0    0    -1
-$EndComp
-Connection ~ 7450 7800
-Wire Wire Line
-	7450 7800 7550 7800
+P 7350 7800
+F 0 "#PWR031" H 7350 7550 50  0001 C CNN
+F 1 "GNDD" H 7354 7645 50  0000 C CNN
+F 2 "" H 7350 7800 50  0001 C CNN
+F 3 "" H 7350 7800 50  0001 C CNN
+	1    7350 7800
+	1    0    0    -1
+$EndComp
+Connection ~ 7350 7800
+Wire Wire Line
+	7350 7800 7550 7800
 $Comp
 L power:+5V #PWR030
@@
 L SamacSys_Parts:HDSP-B03G DS2
 U 1 1 6048D73A
-P 8450 4800
-F 0 "DS2" H 9900 5065 50  0000 C CNN
-F 1 "HDSP-B03G" H 9900 4974 50  0000 C CNN
-F 2 "HDSPB03G" H 11200 4900 50  0001 L CNN
-F 3 "https://docs.broadcom.com/docs/AV01-0698EN" H 11200 4800 50  0001 L CNN
-F 4 "LED Displays & Accessories 88:88 Clock Module 0.56in 4 Digits CC" H 11200 4700 50  0001 L CNN "Description"
-F 5 "8" H 11200 4600 50  0001 L CNN "Height"
-F 6 "630-HDSP-B03G" H 11200 4500 50  0001 L CNN "Mouser Part Number"
-F 7 "https://www.mouser.co.uk/ProductDetail/Broadcom-Avago/HDSP-B03G/?qs=pQfy5%252BKCabJU4dELvEhWiw%3D%3D" H 11200 4400 50  0001 L CNN "Mouser Price/Stock"
-F 8 "Avago Technologies" H 11200 4300 50  0001 L CNN "Manufacturer_Name"
-F 9 "HDSP-B03G" H 11200 4200 50  0001 L CNN "Manufacturer_Part_Number"
-	1    8450 4800
+P 8450 4400
+F 0 "DS2" H 9900 4665 50  0000 C CNN
+F 1 "HDSP-B03G" H 9900 4574 50  0000 C CNN
+F 2 "HDSPB03G" H 11200 4500 50  0001 L CNN
+F 3 "https://docs.broadcom.com/docs/AV01-0698EN" H 11200 4400 50  0001 L CNN
+F 4 "LED Displays & Accessories 88:88 Clock Module 0.56in 4 Digits CC" H 11200 4300 50  0001 L CNN "Description"
+F 5 "8" H 11200 4200 50  0001 L CNN "Height"
+F 6 "630-HDSP-B03G" H 11200 4100 50  0001 L CNN "Mouser Part Number"
+F 7 "https://www.mouser.co.uk/ProductDetail/Broadcom-Avago/HDSP-B03G/?qs=pQfy5%252BKCabJU4dELvEhWiw%3D%3D" H 11200 4000 50  0001 L CNN "Mouser Price/Stock"
+F 8 "Avago Technologies" H 11200 3900 50  0001 L CNN "Manufacturer_Name"
+F 9 "HDSP-B03G" H 11200 3800 50  0001 L CNN "Manufacturer_Part_Number"
+	1    8450 4400
 	1    0    0    -1
 $EndComp
@@
 Text GLabel 5750 4600 0    50   Input ~ 0
 O7
-Text GLabel 5750 4700 0    50   Input ~ 0
-O8
-Wire Wire Line
-	5750 4700 5850 4700
 Wire Wire Line
 	5750 4600 5850 4600
@@
 Wire Wire Line
 	5750 4100 5850 4100
+Wire Wire Line
+	5750 3900 5850 3900
+Text GLabel 11450 3450 2    50   Input ~ 0
+O11
+Text GLabel 11450 4500 2    50   Input ~ 0
+O11
+Wire Wire Line
+	11450 3450 11350 3450
+Wire Wire Line
+	11450 4500 11350 4500
+Text GLabel 8350 3950 0    50   Input ~ 0
+O12
+Wire Wire Line
+	8350 3950 8450 3950
+Text GLabel 8350 5000 0    50   Input ~ 0
+O12
+Wire Wire Line
+	8350 5000 8450 5000
+Text GLabel 8350 3650 0    50   Input ~ 0
+O13
+Wire Wire Line
+	8350 3650 8450 3650
+Text GLabel 8350 4700 0    50   Input ~ 0
+O13
+Wire Wire Line
+	8350 4700 8450 4700
+Text GLabel 8350 4500 0    50   Input ~ 0
+O14
+Wire Wire Line
+	8350 4500 8450 4500
+Text GLabel 8350 3450 0    50   Input ~ 0
+O14
+Wire Wire Line
+	8450 3450 8350 3450
+Text GLabel 8350 3350 0    50   Input ~ 0
+O15
+Wire Wire Line
+	8350 3350 8450 3350
+Text GLabel 8350 4400 0    50   Input ~ 0
+O15
+Wire Wire Line
+	8350 4400 8450 4400
+Text GLabel 11450 4600 2    50   Input ~ 0
+O16
+Wire Wire Line
+	11350 4600 11450 4600
+Text GLabel 11450 3550 2    50   Input ~ 0
+O16
+Wire Wire Line
+	11450 3550 11350 3550
+Text GLabel 8350 3550 0    50   Input ~ 0
+O18
+Wire Wire Line
+	8350 3750 8450 3750
+Text GLabel 8350 4600 0    50   Input ~ 0
+O18
+Wire Wire Line
+	8350 4800 8450 4800
+Wire Wire Line
+	8350 3550 8450 3550
+Wire Wire Line
+	8350 4600 8450 4600
+Text GLabel 8350 3750 0    50   Input ~ 0
+O17
+Text GLabel 8350 4800 0    50   Input ~ 0
+O17
 Text GLabel 5750 3900 0    50   Input ~ 0
 O0
-Wire Wire Line
-	5750 3900 5850 3900
+Text GLabel 11450 3350 2    50   Input ~ 0
+O0
+Wire Wire Line
+	11450 3350 11350 3350
+Text GLabel 11450 3650 2    50   Input ~ 0
+O1
+Wire Wire Line
+	11350 3650 11450 3650
+Text GLabel 11450 3750 2    50   Input ~ 0
+O2
+Wire Wire Line
+	11350 3750 11450 3750
+Text GLabel 8350 3850 0    50   Input ~ 0
+O3
+Wire Wire Line
+	8350 3850 8450 3850
+Text GLabel 11450 4400 2    50   Input ~ 0
+O4
+Wire Wire Line
+	11350 4400 11450 4400
+Text GLabel 11450 4700 2    50   Input ~ 0
+O5
+Wire Wire Line
+	11350 4700 11450 4700
+Text GLabel 11450 4800 2    50   Input ~ 0
+O6
+Wire Wire Line
+	11350 4800 11450 4800
+Text GLabel 8350 4900 0    50   Input ~ 0
+O7
+Wire Wire Line
+	8350 4900 8450 4900
+$Comp
+L power:GNDD #PWR?
+U 1 1 605D0451
+P 5450 3800
+F 0 "#PWR?" H 5450 3550 50  0001 C CNN
+F 1 "GNDD" H 5454 3645 50  0000 C CNN
+F 2 "" H 5450 3800 50  0001 C CNN
+F 3 "" H 5450 3800 50  0001 C CNN
+	1    5450 3800
+	1    0    0    -1
+$EndComp
+Wire Wire Line
+	5450 3800 5850 3800
+Wire Wire Line
+	5850 3500 5450 3500
+Wire Wire Line
+	5450 3500 5450 3800
+Connection ~ 5450 3800
 $EndSCHEMATC

Commit message: Update Schema
Parts:
- added C11, C12: 22nF, symbol Device:C
- added R14, R16: 1k, symbol Device:R
- added R15, R17: 100k, symbol Device:R
- added SW1, SW2: SW_Push, symbol Switch:SW_Push
Connections:
- net labels added: µC
- wire segments 212 -> 230
Changed lines of the file:
@@
 	8350 4900 8450 4900
 $Comp
-L power:GNDD #PWR?
+L power:GNDD #PWR065
 U 1 1 605D0451
 P 5450 3800
-F 0 "#PWR?" H 5450 3550 50  0001 C CNN
+F 0 "#PWR065" H 5450 3550 50  0001 C CNN
 F 1 "GNDD" H 5454 3645 50  0000 C CNN
 F 2 "" H 5450 3800 50  0001 C CNN
@@
 	5450 3500 5450 3800
 Connection ~ 5450 3800
+$Comp
+L Switch:SW_Push SW1
+U 1 1 605ACBDB
+P 10400 8200
+F 0 "SW1" H 10400 8485 50  0000 C CNN
+F 1 "SW_Push" H 10400 8394 50  0000 C CNN
+F 2 "" H 10400 8400 50  0001 C CNN
+F 3 "~" H 10400 8400 50  0001 C CNN
+	1    10400 8200
+	0    -1   -1   0
+$EndComp
+$Comp
+L Device:R R15
+U 1 1 605BE610
+P 10800 7750
+F 0 "R15" H 10870 7796 50  0000 L CNN
+F 1 "100k" H 10870 7705 50  0000 L CNN
+F 2 "" V 10730 7750 50  0001 C CNN
+F 3 "~" H 10800 7750 50  0001 C CNN
+	1    10800 7750
+	1    0    0    -1
+$EndComp
+$Comp
+L Device:R R14
+U 1 1 605C03A8
+P 10600 7950
+F 0 "R14" V 10393 7950 50  0000 C CNN
+F 1 "1k" V 10484 7950 50  0000 C CNN
+F 2 "" V 10530 7950 50  0001 C CNN
+F 3 "~" H 10600 7950 50  0001 C CNN
+	1    10600 7950
+	0    1    1    0
+$EndComp
+Wire Wire Line
+	10400 8000 10400 7950
+Wire Wire Line
+	10400 7950 10450 7950
+Wire Wire Line
+	10750 7950 10800 7950
+Wire Wire Line
+	10800 7950 10800 7900
+$Comp
+L Device:C C11
+U 1 1 605DD994
+P 10800 8200
+F 0 "C11" H 10915 8246 50  0000 L CNN
+F 1 "22nF" H 10915 8155 50  0000 L CNN
+F 2 "" H 10838 8050 50  0001 C CNN
+F 3 "~" H 10800 8200 50  0001 C CNN
+	1    10800 8200
+	1    0    0    -1
+$EndComp
+Wire Wire Line
+	10800 8050 10800 7950
+Connection ~ 10800 7950
+Wire Wire Line
+	10800 8350 10800 8400
+Wire Wire Line
+	10800 8400 10600 8400
+$Comp
+L power:+3V3 #PWR067
+U 1 1 6061981A
+P 10800 7600
+F 0 "#PWR067" H 10800 7450 50  0001 C CNN
+F 1 "+3V3" H 10800 7750 50  0000 C CNN
+F 2 "" H 10800 7600 50  0001 C CNN
+F 3 "" H 10800 7600 50  0001 C CNN
+	1    10800 7600
+	-1   0    0    -1
+$EndComp
+$Comp
+L power:GNDD #PWR066
+U 1 1 60619F83
+P 10600 8400
+F 0 "#PWR066" H 10600 8150 50  0001 C CNN
+F 1 "GNDD" H 10604 8245 50  0000 C CNN
+F 2 "" H 10600 8400 50  0001 C CNN
+F 3 "" H 10600 8400 50  0001 C CNN
+	1    10600 8400
+	-1   0    0    -1
+$EndComp
+Connection ~ 10600 8400
+Wire Wire Line
+	10600 8400 10400 8400
+Text GLabel 11000 7950 2    50   Input ~ 0
+µC
+Wire Wire Line
+	11000 7950 10800 7950
+$Comp
+L Switch:SW_Push SW2
+U 1 1 605AD2CF
+P 11600 8200
+F 0 "SW2" H 11600 8485 50  0000 C CNN
+F 1 "SW_Push" H 11600 8394 50  0000 C CNN
+F 2 "" H 11600 8400 50  0001 C CNN
+F 3 "~" H 11600 8400 50  0001 C CNN
+	1    11600 8200
+	0    -1   -1   0
+$EndComp
+$Comp
+L Device:R R17
+U 1 1 6065FD1A
+P 12000 7750
+F 0 "R17" H 12070 7796 50  0000 L CNN
+F 1 "100k" H 12070 7705 50  0000 L CNN
+F 2 "" V 11930 7750 50  0001 C CNN
+F 3 "~" H 12000 7750 50  0001 C CNN
+	1    12000 7750
+	1    0    0    -1
+$EndComp
+$Comp
+L Device:R R16
+U 1 1 6065FD20
+P 11800 7950
+F 0 "R16" V 11593 7950 50  0000 C CNN
+F 1 "1k" V 11684 7950 50  0000 C CNN
+F 2 "" V 11730 7950 50  0001 C CNN
+F 3 "~" H 11800 7950 50  0001 C CNN
+	1    11800 7950
+	0    1    1    0
+$EndComp
+Wire Wire Line
+	11600 7950 11650 7950
+Wire Wire Line
+	11950 7950 12000 7950
+Wire Wire Line
+	12000 7950 12000 7900
+$Comp
+L Device:C C12
+U 1 1 6065FD29
+P 12000 8200
+F 0 "C12" H 12115 8246 50  0000 L CNN
+F 1 "22nF" H 12115 8155 50  0000 L CNN
+F 2 "" H 12038 8050 50  0001 C CNN
+F 3 "~" H 12000 8200 50  0001 C CNN
+	1    12000 8200
+	1    0    0    -1
+$EndComp
+Wire Wire Line
+	12000 8050 12000 7950
+Connection ~ 12000 7950
+Wire Wire Line
+	12000 8350 12000 8400
+Wire Wire Line
+	12000 8400 11800 8400
+$Comp
+L power:+3V3 #PWR069
+U 1 1 6065FD33
+P 12000 7600
+F 0 "#PWR069" H 12000 7450 50  0001 C CNN
+F 1 "+3V3" H 12000 7750 50  0000 C CNN
+F 2 "" H 12000 7600 50  0001 C CNN
+F 3 "" H 12000 7600 50  0001 C CNN
+	1    12000 7600
+	-1   0    0    -1
+$EndComp
+$Comp
+L power:GNDD #PWR068
+U 1 1 6065FD39
+P 11800 8400
+F 0 "#PWR068" H 11800 8150 50  0001 C CNN
+F 1 "GNDD" H 11804 8245 50  0000 C CNN
+F 2 "" H 11800 8400 50  0001 C CNN
+F 3 "" H 11800 8400 50  0001 C CNN
+	1    11800 8400
+	-1   0    0    -1
+$EndComp
+Connection ~ 11800 8400
+Wire Wire Line
+	11800 8400 11600 8400
+Text GLabel 12200 7950 2    50   Input ~ 0
+µC
+Wire Wire Line
+	12200 7950 12000 7950
+Wire Wire Line
+	11600 8000 11600 7950
 $EndSCHEMATC

Commit message: Update schematic
Parts:
- removed J1: Conn_01x02_MountingPin, symbol Connector_Generic_MountingPin:Conn_01x02_MountingPin
- removed J2, J3: Conn_01x03_MountingPin, symbol Connector_Generic_MountingPin:Conn_01x03_MountingPin
- removed J4: Conn_01x04_MountingPin, symbol Connector_Generic_MountingPin:Conn_01x04_MountingPin
- added C13, C14: 4.7µF, symbol Device:C
- added IC1: ZLDO1117K33TC, TO-252_1, symbol SamacSys_Parts:ZLDO1117K33TC
- added J1: Conn_01x02, symbol Connector_Generic:Conn_01x02
- added J2: Conn_01x06, symbol Connector_Generic:Conn_01x06
- added J3, J6, J7: Conn_01x04, symbol Connector_Generic:Conn_01x04
- added J4, J5: Conn_01x03, symbol Connector_Generic:Conn_01x03
Connections:
- net labels added: CLK, QH, SER, SH
- net labels removed: PB13, PB15
- wire segments 230 -> 244
Other:
- moved on the sheet: C1, C2, L1, R2, R3, R4, U1, U3

Commit message: Update Schematic
Parts:
- removed C1: 10µF, symbol Device:CP
- removed C2: 4,7µF, symbol Device:CP
- removed L1: 10µH, symbol pspice:INDUCTOR
- removed R2: 10k, symbol Device:R
- removed U1: TPS62203DBV, Package_TO_SOT_SMD:SOT-23-5, symbol Regulator_Switching:TPS62203DBV
- removed U3: TXB0102DCU, Package_SO:VSSOP-8_2.4x2.1mm_P0.5mm, symbol Logic_LevelTranslator:TXB0102DCU
- added IC12: SN74LVC2T45DCTRE4, SOP65P400X130-8N, symbol SamacSys_Parts:SN74LVC2T45DCTRE4
- renumbered IC1 to IC13
Connections:
- net +3V3: now also IC12.1 (VCCA), IC12.5 (DIR)
- net +5V: now also IC12.8 (VCCB)
- net GNDD: now also IC12.4 (GND)
- net at U2.34 (PB13): now also IC12.3 (A2)
- net at U2.36 (PB15): now also IC12.2 (A1)
- net at J7.3 (Pin_3): now also IC12.6 (B2)
- net at J7.2 (Pin_2): now also IC12.7 (B1)
Other:
- note added: "Boot Modes\n\n"
- note added: "Switch \n"
- moved on the sheet: C10, C11, C12, C13, C14, C7, C8, C9, D1, D2, D3, D4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
