File: Schaakbord/Schaakbord.sch (KiCad schematic (older format))
At the start: 61 parts, among them IC1 ZLDO1117K33TC, IC10 AH3572-SA-7, IC11 MAX6955AAX+, IC12 SN74LVC2T45DCTRE4, IC13 M24C04-RMN6TP, IC2 SN74HC165DR, IC3 AH3572-SA-7, IC4 AH3572-SA-7, IC5 AH3572-SA-7, IC6 AH3572-SA-7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

Commit message: Update Schematic
Parts:
- added C1, C2: 12µF, symbol Device:C_Small
- added C15: 0.1µF, symbol Device:C_Small
- added R2: 10k, symbol Device:R_Small
Connections:
- net +3V3: now also C1.2, C15.2, R2.1; no longer IC12.5 (DIR)
- net +5V: now also C2.1
- net GNDD: now also C1.1, C15.1, C2.2
- new net: IC12.5 (DIR), R2.2
Changed lines of the file:
@@
 Connection ~ 5500 8850
 Wire Wire Line
-	4750 8900 5150 8900
-Wire Wire Line
-	5150 8900 5150 8300
-Wire Wire Line
-	5150 8300 5500 8300
+	4750 8900 5200 8900
+Wire Wire Line
+	5200 8900 5200 8300
+Wire Wire Line
+	5200 8300 5500 8300
 Connection ~ 5500 8300
 $Comp
 L power:+3V3 #PWR061
 U 1 1 60468487
-P 4750 8700
-F 0 "#PWR061" H 4750 8550 50  0001 C CNN
-F 1 "+3V3" H 4750 8850 50  0000 C CNN
-F 2 "" H 4750 8700 50  0001 C CNN
-F 3 "" H 4750 8700 50  0001 C CNN
-	1    4750 8700
+P 4750 8450
+F 0 "#PWR061" H 4750 8300 50  0001 C CNN
+F 1 "+3V3" H 4750 8600 50  0000 C CNN
+F 2 "" H 4750 8450 50  0001 C CNN
+F 3 "" H 4750 8450 50  0001 C CNN
+	1    4750 8450
 	-1   0    0    -1
 $EndComp
@@
 	4850 8800 4850 8700
 Wire Wire Line
-	4850 8700 4950 8700
+	4850 8700 4900 8700
 $Comp
 L power:GNDD #PWR060
@@
 U 1 1 604B302F
 P 11400 8750
-F 0 "C8" V 11250 8650 50  0000 C CNN
-F 1 "12pF" V 11250 8850 50  0000 C CNN
+F 0 "C8" V 11150 8750 50  0000 C CNN
+F 1 "12pF" V 11250 8750 50  0000 C CNN
 F 2 "" H 11438 8600 50  0001 C CNN
 F 3 "~" H 11400 8750 50  0001 C CNN
@@
 Wire Wire Line
 	3150 4400 3150 4500
-$Comp
-L power:+3V3 #PWR035
-U 1 1 60910B1C
-P 4400 4950
-F 0 "#PWR035" H 4400 4800 50  0001 C CNN
-F 1 "+3V3" H 4400 5100 50  0000 C CNN
-F 2 "" H 4400 4950 50  0001 C CNN
-F 3 "" H 4400 4950 50  0001 C CNN
-	1    4400 4950
-	1    0    0    -1
-$EndComp
-Wire Wire Line
-	4400 4950 4250 4950
-Wire Wire Line
-	4250 4950 4250 4800
 Wire Wire Line
 	4550 4700 4250 4700
@@
 Text Notes 8900 1200 0    150  ~ 0
 Boot Modes\n\n
+$Comp
+L Device:C_Small C1
+U 1 1 607573C6
+P 3650 5300
+F 0 "C1" H 3900 5250 50  0000 R CNN
+F 1 "12µF" H 3950 5350 50  0000 R CNN
+F 2 "" H 3650 5300 50  0001 C CNN
+F 3 "~" H 3650 5300 50  0001 C CNN
+	1    3650 5300
+	-1   0    0    1
+$EndComp
+$Comp
+L Device:C_Small C2
+U 1 1 6075A611
+P 3850 5300
+F 0 "C2" H 3942 5346 50  0000 L CNN
+F 1 "12µF" H 3942 5255 50  0000 L CNN
+F 2 "" H 3850 5300 50  0001 C CNN
+F 3 "~" H 3850 5300 50  0001 C CNN
+	1    3850 5300
+	1    0    0    -1
+$EndComp
+$Comp
+L power:GNDD #PWR01
+U 1 1 6075C621
+P 3650 5400
+F 0 "#PWR01" H 3650 5150 50  0001 C CNN
+F 1 "GNDD" H 3654 5245 50  0000 C CNN
+F 2 "" H 3650 5400 50  0001 C CNN
+F 3 "" H 3650 5400 50  0001 C CNN
+	1    3650 5400
+	1    0    0    -1
+$EndComp
+$Comp
+L power:GNDD #PWR02
+U 1 1 6075CB99
+P 3850 5400
+F 0 "#PWR02" H 3850 5150 50  0001 C CNN
+F 1 "GNDD" H 3854 5245 50  0000 C CNN
+F 2 "" H 3850 5400 50  0001 C CNN
+F 3 "" H 3850 5400 50  0001 C CNN
+	1    3850 5400
+	1    0    0    -1
+$EndComp
+Text GLabel 3150 4450 0    50   Input ~ 0
+VCCA
+Text GLabel 4250 4500 2    50   Input ~ 0
+VCCB
+Text GLabel 3650 5200 1    50   Input ~ 0
+VCCA
+Text GLabel 3850 5200 1    50   Input ~ 0
+VCCB
+$Comp
+L Device:R_Small R2
+U 1 1 6077E968
+P 4250 4950
+F 0 "R2" H 4191 4904 50  0000 R CNN
+F 1 "10k" H 4191 4995 50  0000 R CNN
+F 2 "" H 4250 4950 50  0001 C CNN
+F 3 "~" H 4250 4950 50  0001 C CNN
+	1    4250 4950
+	-1   0    0    1
+$EndComp
+$Comp
+L power:+3V3 #PWR035
+U 1 1 60910B1C
+P 4100 5100
+F 0 "#PWR035" H 4100 4950 50  0001 C CNN
+F 1 "+3V3" H 4100 5250 50  0000 C CNN
+F 2 "" H 4100 5100 50  0001 C CNN
+F 3 "" H 4100 5100 50  0001 C CNN
+	1    4100 5100
+	1    0    0    -1
+$EndComp
+Wire Wire Line
+	4250 5100 4100 5100
+Wire Wire Line
+	4250 5100 4250 5050
+Wire Wire Line
+	4250 4850 4250 4800
+$Comp
+L Device:C_Small C15
+U 1 1 607CBE31
+P 4900 8600
+F 0 "C15" H 4808 8554 50  0000 R CNN
+F 1 "0.1µF" H 4850 8650 50  0000 R CNN
+F 2 "" H 4900 8600 50  0001 C CNN
+F 3 "~" H 4900 8600 50  0001 C CNN
+	1    4900 8600
+	-1   0    0    1
+$EndComp
+Wire Wire Line
+	4750 8700 4750 8500
+Connection ~ 4900 8700
+Wire Wire Line
+	4900 8700 4950 8700
+Wire Wire Line
+	4900 8500 4750 8500
+Connection ~ 4750 8500
+Wire Wire Line
+	4750 8500 4750 8450
 $EndSCHEMATC

Commit message: Schematic Update
Parts:
- removed C13, C14: 4.7µF, symbol Device:C
- removed IC1: ZLDO1117K33TC, TO-252_1, symbol SamacSys_Parts:ZLDO1117K33TC
- added C16, C17: 10µF, symbol Device:C
- added R18: 10k, symbol Device:R_Small
- added R19: 10, symbol Device:R_Small
- added U1: AP7362, Package_SO:Diodes_SO-8EP, symbol SamacSys_Parts:AP7362
Connections:
- net +3V3: now also C10.1, C9.2, IC11.19 (V+_1), IC11.21 (V+_2), C17.1, R18.1, R19.2, U1.5 (OUT), U1.6 (OUT), U1.7 (OUT)
- net +5V: now also C16.2, U1.2 (EN), U1.3 (IN), U1.4 (IN)
- net PB10: now also R18.2
- net PB11: now also R19.1
- net GNDD renamed GND
- net GND: now also C16.1, C17.2, U1.1 (GND), U1.9 (GND)
Other:
- moved on the sheet: C10, C8, C9
