File: Schaakbord/Hoofdbord/Hoofdbord.sch (KiCad schematic (older format))
At the start: 41 parts, among them IC1 SN74LVC2T45DCTRE4, IC2 M24C04-RMN6TP, IC3 MAX6955AAX+, IC4 AP7362, J1 Conn_01x04, J2 Conn_01x03, J3 Conn_01x03, J4 Conn_01x02, SW1 SW_Push, SW2 SW_Push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

Commit message: Schematic Update
Parts:
- C7: value 12pF -> 22pF
- R10: value 110k -> 56k
Changed lines of the file:
@@
 P 7800 4900
 F 0 "R10" V 7750 5100 50  0000 C CNN
-F 1 "110k" V 7850 5100 50  0000 C CNN
+F 1 "56k" V 7850 5100 50  0000 C CNN
 F 2 "Capacitor_SMD:C_0805_2012Metric_Pad1.18x1.45mm_HandSolder" V 7730 4900 50  0001 C CNN
 F 3 "~" H 7800 4900 50  0001 C CNN
@@
 P 9650 5250
 F 0 "C7" H 9450 5200 50  0000 C CNN
-F 1 "12pF" H 9450 5300 50  0000 C CNN
+F 1 "22pF" H 9450 5300 50  0000 C CNN
 F 2 "Capacitor_SMD:C_0805_2012Metric_Pad1.18x1.45mm_HandSolder" H 9688 5100 50  0001 C CNN
 F 3 "~" H 9650 5250 50  0001 C CNN

Commit message: PCB
Parts:
- removed IC4: AP7362, Package_SO:Diodes_SO-8EP, symbol SamacSys_Parts:AP7362
- removed J2, J3: Conn_01x03, Connector_PinHeader_2.54mm:PinHeader_1x03_P2.54mm_Vertical, symbol Connector_Generic:Conn_01x03
- added C14: 1µF, Capacitor_SMD:C_0805_2012Metric_Pad1.18x1.45mm_HandSolder, symbol Device:C
- added C15: 100nF, Capacitor_SMD:C_0805_2012Metric_Pad1.18x1.45mm_HandSolder, symbol Device:C
- added C9: 10µF, Capacitor_SMD:C_0805_2012Metric_Pad1.18x1.45mm_HandSolder, symbol Device:C
- added J3: Rotary_Encoder, Connector_PinHeader_2.54mm:PinHeader_1x05_P2.54mm_Vertical, symbol Connector_Generic:Conn_01x05
- added J4: SWD, Connector_PinHeader_2.54mm:PinHeader_1x04_P2.54mm_Vertical, symbol Connector_Generic:Conn_01x04
- added R14, R15: 10k, Resistor_SMD:R_0805_2012Metric_Pad1.20x1.40mm_HandSolder, symbol Device:R
- added SW3: Boot Modes, SamacSys_Parts:418117270902, symbol Switch:SW_DIP_x02
- added U2: NCP1117-3.3_TO252, Package_TO_SOT_SMD:TO-252-2, symbol Regulator_Linear:NCP1117-3.3_TO252
- C1: renamed from C3; value 20pF -> 22pF
- C2: renamed from C1; value 12µF -> 1µF
- C3: renamed from C2; value 12µF -> 1µF
- C4, C5: value 22nF -> 100nF
- J1: value Conn_01x04 -> APA102C
- J2: renamed from J4; value Conn_01x02 -> 5V_Power
- R1, R2: footprint Capacitor_SMD:C_0805_2012Metric_Pad1.18x1.45mm_HandSolder -> Resistor_SMD:R_0805_2012Metric_Pad1.20x1.40mm_HandSolder
- R10: renamed from R6; value 1k -> 10k; footprint Capacitor_SMD:C_0805_2012Metric_Pad1.18x1.45mm_HandSolder -> Resistor_SMD:R_0805_2012Metric_Pad1.20x1.40mm_HandSolder
- R11: renamed from R9; footprint Capacitor_SMD:C_0805_2012Metric_Pad1.18x1.45mm_HandSolder -> Resistor_SMD:R_0805_2012Metric_Pad1.20x1.40mm_HandSolder
- R12: renamed from R10; footprint Capacitor_SMD:C_0805_2012Metric_Pad1.18x1.45mm_HandSolder -> Resistor_SMD:R_0805_2012Metric_Pad1.20x1.40mm_HandSolder
- R13: renamed from R12; footprint Capacitor_SMD:C_0805_2012Metric_Pad1.18x1.45mm_HandSolder -> Resistor_SMD:R_0805_2012Metric_Pad1.20x1.40mm_HandSolder
- R16: renamed from R11; footprint Capacitor_SMD:C_0805_2012Metric_Pad1.18x1.45mm_HandSolder -> Resistor_SMD:R_0805_2012Metric_Pad1.20x1.40mm_HandSolder
- R3: renamed from R14; footprint Capacitor_SMD:C_0805_2012Metric_Pad1.18x1.45mm_HandSolder -> Resistor_SMD:R_0805_2012Metric_Pad1.20x1.40mm_HandSolder
- R4: renamed from R13; footprint Capacitor_SMD:C_0805_2012Metric_Pad1.18x1.45mm_HandSolder -> Resistor_SMD:R_0805_2012Metric_Pad1.20x1.40mm_HandSolder
- R5: renamed from R3; footprint Capacitor_SMD:C_0805_2012Metric_Pad1.18x1.45mm_HandSolder -> Resistor_SMD:R_0805_2012Metric_Pad1.20x1.40mm_HandSolder
- R6: renamed from R5; value 100k -> 10k; footprint Capacitor_SMD:C_0805_2012Metric_Pad1.18x1.45mm_HandSolder -> Resistor_SMD:R_0805_2012Metric_Pad1.20x1.40mm_HandSolder
- R7: renamed from R4; value 1k -> 10k; footprint Capacitor_SMD:C_0805_2012Metric_Pad1.18x1.45mm_HandSolder -> Resistor_SMD:R_0805_2012Metric_Pad1.20x1.40mm_HandSolder
- R8: value 100k -> 10k; footprint Capacitor_SMD:C_0805_2012Metric_Pad1.18x1.45mm_HandSolder -> Resistor_SMD:R_0805_2012Metric_Pad1.20x1.40mm_HandSolder
- R9: renamed from R7; footprint Capacitor_SMD:C_0805_2012Metric_Pad1.18x1.45mm_HandSolder -> Resistor_SMD:R_0805_2012Metric_Pad1.20x1.40mm_HandSolder
- renumbered C9 to C10, C10 to C11, C11 to C12, C12 to C13, C13 to C16, C14 to C17
Connections:
- net VDD1 is gone; now on net +3V3: C11.2, U1.32 (VDD)
- net VDD2 is gone; now on net +3V3: C12.2, U1.48 (VDD)
- net VDD3 is gone; now on net +3V3: C13.2, U1.64 (VDD)
- net VDD4 is gone; now on net +3V3: C10.2, U1.19 (VDD)
- net VSS1 is gone; now on net GNDD: C11.1, U1.31 (VSS)
- net VSS2 is gone; now on net GNDD: C12.1, U1.47 (VSS)
- net VSS3 is gone; now on net GNDD: C13.1, U1.63 (VSS)
- net VSS4 is gone; now on net GNDD: C10.1, U1.18 (VSS)
- net +3V3: now also R3.2, R6.2, R8.2, C14.2, C15.2, C9.2, J4.1 (Pin_1), R14.2, R15.1, U2.2 (VO); no longer R3.1, R6.1, R8.1
- net +5V: now also J3.1 (Pin_1), U2.3 (VI)
- net µC: no longer R6.2, R8.2
- net PA0: now reaches U1.14 (PA0)
- net PA0: now also J3.2 (Pin_2)
- net PA1: now reaches U1.15 (PA1)
- net PA1: now also J3.3 (Pin_3)
- net PA2: now reaches U1.16 (PA2)
- net PA2: now also J3.4 (Pin_4)
- net PB13: now reaches IC1.3 (A2), U1.34 (PB13)
- net PB13: now also R3.1; no longer R3.2
- net PB15: now reaches IC1.2 (A1), R4.1, U1.36 (PB15)
- net PA13: now reaches U1.46 (PA13)
- net PA13: now also J4.3 (Pin_3)
- net PA14: now reaches U1.49 (PA14)
- net PA14: now also J4.2 (Pin_2)
- net at R16.1: now also R15.2, SW3.3
- net at R13.1: now also R14.1, SW3.4
- net at R7.2, SW1.2: now also R6.1
- net at R10.2, SW2.2: now also R8.1
- net GND renamed GNDD
- net GNDD: now also C14.1, C15.1, C9.1, J3.5 (Pin_5), J4.4 (Pin_4), SW3.1, SW3.2, U2.1 (GND)
Other:
- moved on the sheet: C10, C11, C12, C13, C2, C3, C4, C5, IC1, J1, R10, R13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

Commit message: Schematic Update
Connections:
- net +3V3: now also J3.5 (Pin_5), J4.4 (Pin_4); no longer J4.1 (Pin_1)
- net +5V: now also J1.4 (Pin_4), J2.2 (Pin_2); no longer J1.1 (Pin_1), J2.1 (Pin_1), J3.1 (Pin_1)
- net GNDD: now also J1.1 (Pin_1), J2.1 (Pin_1), J3.1 (Pin_1), J4.1 (Pin_1); no longer J1.4 (Pin_4), J2.2 (Pin_2), J3.5 (Pin_5), J4.4 (Pin_4)
- net PA0: now also J3.4 (Pin_4); no longer J3.2 (Pin_2)
- net PA13: now also J4.2 (Pin_2); no longer J4.3 (Pin_3)
- net PA14: now also J4.3 (Pin_3); no longer J4.2 (Pin_2)
- net PA2: now also J3.2 (Pin_2); no longer J3.4 (Pin_4)
- net PC0: now reaches U1.8 (PC0)
- net PC0: now also C4.1, R7.1
- net PC1: now reaches U1.9 (PC1)
- net PC1: now also C5.1, R10.1
- net at IC1.6 (B2): now also J1.2 (Pin_2); no longer J1.3 (Pin_3)
- net at IC1.7 (B1): now also J1.3 (Pin_3); no longer J1.2 (Pin_2)
- removed net µC: C4.1, C5.1, R10.1, R7.1
