File: Schaakbord/Hoofdbord/Hoofdbord.kicad_pcb (KiCad board)
At the start: 2 copper layers, 41 parts, among them IC1 SN74LVC2T45DCTRE4, IC2 M24C04-RMN6TP, IC3 MAX6955AAX+, IC4 AP7362, J1 Conn_01x04, J2 Conn_01x03, J3 Conn_01x03, J4 Conn_01x02, SW1 SW_Push, SW2 SW_Push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

Commit message: Schematic Update
Parts:
- moved IC3 49.0 mm to (166.6, 57.8), turned to 90 degrees
- moved R7 44.3 mm to (162.2, 64.8)
- moved R9 41.2 mm to (161.2, 66.8), turned to 180 degrees
- moved R12 40.0 mm to (147.1, 65.6), turned to 270 degrees
- moved J3 38.6 mm to (144.1, 62.1)
- moved C7 38.4 mm to (173.6, 50.8), turned to 180 degrees
- moved SW2 38.3 mm to (176.0, 95.0)
- moved R10 35.8 mm to (173.7, 64.6)
- moved C6 29.2 mm to (176.6, 56.6), turned to 180 degrees
- moved J4 26.0 mm to (171.8, 32.1)
- moved R8 23.5 mm to (180.3, 110.9)
- moved C4 23.0 mm to (170.2, 113.5)
- moved R4 20.6 mm to (172.2, 103.0)
- moved C8 20.0 mm to (176.6, 58.7)
- moved R11 18.5 mm to (151.5, 86.9)
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Routing:
- net GND: track 25.6 -> 49.1 mm
- net +3V3: track 15.7 -> 30.0 mm
- net PB10: track 0.00 -> 9.10 mm
- net PB11: track 0.00 -> 8.78 mm
- net Net-(C7-Pad2): track 0.00 -> 2.26 mm
- net Net-(IC3-Pad17): track 0.00 -> 2.13 mm

Commit message: PCB
Parts:
- removed the C13 at (156.8, 39.1)
- removed IC4: AP7362, Package_SO:Diodes_SO-8EP
- added C15: 100nF, Capacitor_SMD:C_0805_2012Metric_Pad1.18x1.45mm_HandSolder, F.Cu at (172.7, 78.7)
- added C16: 10µF, Capacitor_SMD:C_0805_2012Metric_Pad1.18x1.45mm_HandSolder, F.Cu at (146.9, 64.9)
- added C17: 10µF, Capacitor_SMD:C_0805_2012Metric_Pad1.18x1.45mm_HandSolder, F.Cu at (150.5, 59.2)
- added C9: 10µF, Capacitor_SMD:C_0805_2012Metric_Pad1.18x1.45mm_HandSolder, F.Cu at (172.1, 69.7)
- added R15: 10k, Resistor_SMD:R_0805_2012Metric_Pad1.20x1.40mm_HandSolder, F.Cu at (184.3, 70.5)
- added R16: 10k, Resistor_SMD:R_0805_2012Metric_Pad1.20x1.40mm_HandSolder, F.Cu at (187.2, 71.6)
- added SW3: Boot Modes, SamacSys_Parts:418117270902, F.Cu at (181.7, 82.5)
- added U2: NCP1117-3.3_TO252, Package_TO_SOT_SMD:TO-252-2, F.Cu at (153.6, 63.6)
- C1: renamed from C3; value 20pF -> 22pF
- C14: value 10µF -> 1µF
- C2: renamed from C1; value 12µF -> 1µF
- C3: renamed from C2; value 12µF -> 1µF
- C4, C5: value 22nF -> 100nF
- C7: value 12pF -> 22pF
- J1: value Conn_01x04 -> APA102C
- J2: value Conn_01x03 -> 5V_Power; footprint Connector_PinHeader_2.54mm:PinHeader_1x03_P2.54mm_Vertical -> Connector_PinHeader_2.54mm:PinHeader_1x02_P2.54mm_Vertical
- J3: value Conn_01x03 -> Rotary_Encoder; footprint Connector_PinHeader_2.54mm:PinHeader_1x03_P2.54mm_Vertical -> Connector_PinHeader_2.54mm:PinHeader_1x05_P2.54mm_Vertical
- J4: value Conn_01x02 -> SWD; footprint Connector_PinHeader_2.54mm:PinHeader_1x02_P2.54mm_Vertical -> Connector_PinHeader_2.54mm:PinHeader_1x04_P2.54mm_Vertical
- R1, R11, R13, R14, R2, R3, R7, R9: footprint Capacitor_SMD:C_0805_2012Metric_Pad1.18x1.45mm_HandSolder -> Resistor_SMD:R_0805_2012Metric_Pad1.20x1.40mm_HandSolder
- R10: value 110k -> 10k; footprint Capacitor_SMD:C_0805_2012Metric_Pad1.18x1.45mm_HandSolder -> Resistor_SMD:R_0805_2012Metric_Pad1.20x1.40mm_HandSolder
- R12: value 10k -> 56k; footprint Capacitor_SMD:C_0805_2012Metric_Pad1.18x1.45mm_HandSolder -> Resistor_SMD:R_0805_2012Metric_Pad1.20x1.40mm_HandSolder
- R4, R6: value 1k -> 10k; footprint Capacitor_SMD:C_0805_2012Metric_Pad1.18x1.45mm_HandSolder -> Resistor_SMD:R_0805_2012Metric_Pad1.20x1.40mm_HandSolder
- R5, R8: value 100k -> 10k; footprint Capacitor_SMD:C_0805_2012Metric_Pad1.18x1.45mm_HandSolder -> Resistor_SMD:R_0805_2012Metric_Pad1.20x1.40mm_HandSolder
- moved DS2 98.5 mm to (108.0, 82.5)
- moved J4 63.6 mm to (144.1, 89.3), turned to 180 degrees
- moved R8 53.7 mm to (161.5, 60.6), turned to 90 degrees
- moved C4 52.0 mm to (172.1, 61.6)
- moved R5 49.5 mm to (149.4, 71.6), turned to 180 degrees
- moved C5 48.9 mm to (168.3, 59.1), turned to 180 degrees
- moved R12 44.7 mm to (190.1, 77.9)
- moved R6 43.1 mm to (178.8, 60.1), turned to 270 degrees
- moved R11 42.2 mm to (187.9, 65.5), turned to 90 degrees
- moved SW1 40.9 mm to (175.9, 61.6), turned to 180 degrees
- moved C7 40.1 mm to (200.2, 80.9), turned to 90 degrees
- moved SW2 37.8 mm to (164.5, 59.1)
- moved J3 37.2 mm to (175.5, 82.0), turned to 180 degrees
- moved IC3 33.0 mm to (196.9, 70.9), turned to 0 degrees
- moved C14 32.9 mm to (172.7, 75.0), turned to 90 degrees
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- renumbered C9 to C10, C10 to C11, C11 to C12, C12 to C13
Connections:
- C10 pad 1: VSS4 -> GND
- C10 pad 2: VDD4 -> +3V3
- C11 pad 1: VSS1 -> GND
- C11 pad 2: VDD1 -> +3V3
- C12 pad 1: VSS2 -> GND
- C12 pad 2: VDD2 -> +3V3
- C13 pad 1: VSS3 -> GND
- C13 pad 2: VDD3 -> +3V3
- C14 pad 1: +3V3 -> GND
- C14 pad 2: GND -> +3V3
- IC1 pad 2: Net-(IC1-Pad2) -> PB15
- IC1 pad 3: Net-(IC1-Pad3) -> PB13
- J2 pad 1: +3V3 -> +5V
- J2 pad 2: Net-(J2-Pad2) -> GND
- J3 pad 1: +3V3 -> +5V
- J3 pad 2: Net-(J3-Pad2) -> PA0
- J3 pad 3: GND -> PA1
- J4 pad 1: +5V -> +3V3
- J4 pad 2: GND -> PA14
- R10 pad 1: Net-(IC3-Pad17) -> µC
- R10 pad 2: GND -> Net-(R10-Pad2)
- R11 pad 1: Net-(J2-Pad2) -> PB11
- R11 pad 2: BOOT0 -> +3V3
- R12 pad 1: Net-(J3-Pad2) -> Net-(IC3-Pad17)
- R12 pad 2: BOOT1 -> GND
- R13 pad 1: Net-(IC1-Pad2) -> Net-(R13-Pad1)
- R13 pad 2: +3V3 -> BOOT1
- R14 pad 1: +3V3 -> Net-(R13-Pad1)
- R14 pad 2: Net-(IC1-Pad3) -> +3V3
- R3 pad 1: +3V3 -> PB13
- R3 pad 2: Net-(IC1-Pad5) -> +3V3
- R4 pad 1: µC -> PB15
- R4 pad 2: Net-(R4-Pad2) -> +3V3
- R5 pad 2: µC -> Net-(IC1-Pad5)
- R6 pad 1: µC -> Net-(R6-Pad1)
- R6 pad 2: Net-(R6-Pad2) -> +3V3
- R7 pad 1: +3V3 -> µC
- R7 pad 2: PB10 -> Net-(R6-Pad1)
- R8 pad 1: +3V3 -> Net-(R10-Pad2)
- R8 pad 2: µC -> +3V3
- R9 pad 1: PB11 -> +3V3
- R9 pad 2: +3V3 -> PB10
- SW1 pad 2: Net-(R4-Pad2) -> Net-(R6-Pad1)
- SW2 pad 2: Net-(R6-Pad2) -> Net-(R10-Pad2)
- U1 pad 14: Net-(U1-Pad14) -> PA0
- U1 pad 15: Net-(U1-Pad15) -> PA1
- U1 pad 16: Net-(U1-Pad16) -> PA2
- U1 pad 18: VSS4 -> GND
- U1 pad 19: VDD4 -> +3V3
- U1 pad 31: VSS1 -> GND
- U1 pad 32: VDD1 -> +3V3
- U1 pad 34: Net-(IC1-Pad3) -> PB13
- U1 pad 36: Net-(IC1-Pad2) -> PB15
- U1 pad 46: Net-(U1-Pad46) -> PA13
- U1 pad 47: VSS2 -> GND
- U1 pad 48: VDD2 -> +3V3
- U1 pad 49: Net-(U1-Pad49) -> PA14
- U1 pad 63: VSS3 -> GND
- U1 pad 64: VDD3 -> +3V3
Routing:
- net GND: track 49.1 -> 282.8 mm, vias 12 -> 4
- net +3V3: track 30.0 -> 246.9 mm, vias 0 -> 8
- net O17: track 0.00 -> 137.5 mm
- net O11: track 0.00 -> 136.5 mm
- net O16: track 0.00 -> 136.4 mm
- net O13: track 0.00 -> 135.1 mm
- net O14: track 0.00 -> 129.7 mm
- net O18: track 0.00 -> 128.9 mm
- net O15: track 0.00 -> 123.8 mm
- net O12: track 0.00 -> 123.5 mm
- net O4: track 0.00 -> 95.3 mm, vias 0 -> 1
- net O7: track 0.00 -> 94.8 mm, vias 0 -> 1
- net O5: track 0.00 -> 86.1 mm, vias 0 -> 1
- net O6: track 0.00 -> 82.8 mm, vias 0 -> 1
- net +5V: track 7.29 -> 68.5 mm
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- removed copper zone on B.Cu, net GND

Commit message: Update PCB
Routing:
- net GND: track 282.8 -> 259.3 mm, vias 4 -> 2
- net PA14: track 18.7 -> 20.4 mm
- net PA13: track 18.3 -> 17.1 mm
- net O12: track 123.5 -> 124.4 mm
- net O5: track 86.1 -> 85.5 mm

Commit message: Schematic Update
Parts:
- added ?: MountingHole_3.2mm_M3_Pad_Via, MountingHole:MountingHole_3.2mm_M3_Pad_Via, F.Cu at (94.1, 59.8)
- added ?: MountingHole_3.2mm_M3_Pad_Via, MountingHole:MountingHole_3.2mm_M3_Pad_Via, F.Cu at (236.1, 90.7)
- added ?: MountingHole_3.2mm_M3_Pad_Via, MountingHole:MountingHole_3.2mm_M3_Pad_Via, F.Cu at (94.1, 90.7)
- added ?: MountingHole_3.2mm_M3_Pad_Via, MountingHole:MountingHole_3.2mm_M3_Pad_Via, F.Cu at (236.1, 59.8)
- J1, J2, J3, J4, SW1, SW2: moved to B.Cu
- moved SW2 36.9 mm to (193.2, 82.3), turned to 90 degrees
- moved R8 31.7 mm to (183.4, 83.6)
- moved C5 29.3 mm to (187.1, 81.6), turned to 90 degrees
- moved R10 27.8 mm to (185.3, 83.6), turned to 270 degrees
- moved SW1 25.9 mm to (177.2, 87.5), turned to 270 degrees
- moved R7 25.7 mm to (179.6, 83.6), turned to 270 degrees
- moved R6 23.7 mm to (181.5, 83.6), turned to 90 degrees
- moved C4 22.6 mm to (177.7, 83.5), turned to 270 degrees
- moved J3 9.91 mm to (175.3, 72.1)
- moved C14 9.89 mm to (172.0, 84.8)
- moved J1 7.24 mm to (144.0, 71.2)
- moved J4 7.05 mm to (143.9, 82.3), turned to 270 degrees
- moved R2 6.26 mm to (163.0, 85.3), turned to 180 degrees
- moved C1 4.11 mm to (157.1, 90.4)
- moved IC2 4.04 mm to (155.4, 86.6)
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Connections:
- C4 pad 1: µC -> PC0
- C5 pad 1: µC -> PC1
- J1 pad 1: +5V -> GND
- J1 pad 2: Net-(IC1-Pad7) -> Net-(IC1-Pad6)
- J1 pad 3: Net-(IC1-Pad6) -> Net-(IC1-Pad7)
- J1 pad 4: GND -> +5V
- J2 pad 1: +5V -> GND
- J2 pad 2: GND -> +5V
- J3 pad 1: +5V -> GND
- J3 pad 2: PA0 -> PA2
- J3 pad 4: PA2 -> PA0
- J3 pad 5: GND -> +3V3
- J4 pad 1: +3V3 -> GND
- J4 pad 2: PA14 -> PA13
- J4 pad 3: PA13 -> PA14
- J4 pad 4: GND -> +3V3
- R10 pad 1: µC -> PC1
- R7 pad 1: µC -> PC0
- U1 pad 8: Net-(U1-Pad8) -> PC0
- U1 pad 9: Net-(U1-Pad9) -> PC1
Routing:
- net GND: track 259.3 -> 292.4 mm, vias 2 -> 3
- net +5V: track 68.5 -> 35.6 mm
- net PC1: track 0.00 -> 18.7 mm
- net +3V3: track 246.8 -> 230.1 mm, vias 8 -> 7
- net PC0: track 0.00 -> 11.8 mm
- net BOOT0: track 30.5 -> 41.7 mm, vias 0 -> 2
- net PA14: track 20.4 -> 12.6 mm
- net µC: track 5.09 -> 0.00 mm
- net PB6: track 13.4 -> 9.40 mm
- net PB7: track 16.1 -> 13.3 mm
- net Net-(R10-Pad2): track 5.73 -> 8.19 mm
- net PA13: track 17.1 -> 14.7 mm, vias 1 -> 0
- net Net-(IC1-Pad5): track 1.91 -> 3.51 mm
- net O14: track 129.7 -> 128.2 mm
- net O18: track 128.9 -> 127.3 mm
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- added copper zone on B.Cu, net GND
- added copper zone on F.Cu, net GND
Other:
- board outline added: 150.1 x 39 mm

Commit message: Ontwerp Update
Parts:
- removed the ? at (94.1, 59.8)
- removed the ? at (236.1, 90.7)
- removed the ? at (94.1, 90.7)
- removed the ? at (236.1, 59.8)
- added ?: MountingHole_3.2mm_M3_Pad_Via, MountingHole:MountingHole_3.2mm_M3_Pad_Via, F.Cu at (-71.9, -15.5)
- added ?: MountingHole_3.2mm_M3_Pad_Via, MountingHole:MountingHole_3.2mm_M3_Pad_Via, F.Cu at (70.0, 15.4)
- added ?: MountingHole_3.2mm_M3_Pad_Via, MountingHole:MountingHole_3.2mm_M3_Pad_Via, F.Cu at (-71.9, 15.4)
- added ?: MountingHole_3.2mm_M3_Pad_Via, MountingHole:MountingHole_3.2mm_M3_Pad_Via, F.Cu at (70.0, -15.5)
- moved C17 184.9 mm to (-19.4, -13.6), turned to 270 degrees
- moved C12 182.3 mm to (-8.42, 7.37)
- moved C14 182.3 mm to (5.91, 9.50)
- moved C16 182.3 mm to (-19.3, -9.78)
- moved C3 182.3 mm to (-17.7, 2.54)
- moved C4 182.3 mm to (11.6, 8.23)
- moved C5 182.3 mm to (21.0, 6.24)
- moved C7 182.3 mm to (34.0, 6.20)
- moved C8 182.3 mm to (29.8, 6.18)
- moved C9 182.3 mm to (5.91, -4.97)
- moved DS1 182.3 mm to (40.8, 7.87)
- moved DS2 182.3 mm to (-58.2, 7.87)
- moved J1 182.3 mm to (-22.0, -4.06)
- moved J2 182.3 mm to (-22.1, -11.3)
- moved R10 182.3 mm to (19.2, 8.27)
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Routing:
- net GND: track 292.4 -> 558.0 mm
- net +3V3: track 230.1 -> 241.1 mm, vias 7 -> 8
Other:
- board text added: "Schaakbord M.H."
