File: Schaakbord/Bord/Schaakbord_Bord.kicad_pcb (KiCad board)
At the start: 2 copper layers, 38 parts, among them IC1 SN74HC165DR, IC2 AH3572-SA-7, IC3 AH3572-SA-7, IC4 AH3572-SA-7, IC5 AH3572-SA-7, IC6 AH3572-SA-7, IC7 AH3572-SA-7, IC8 AH3572-SA-7, IC9 AH3572-SA-7, J1 Conn_01x06, J2 Conn_01x06, J3 Conn_01x04, J4 Conn_01x04

Commit message: PCB
Parts:
- added JP1: Jumper, Jumper:SolderJumper-2_P1.3mm_Open_TrianglePad1.0x1.5mm, B.Cu at (155.4, -13.7)
- C5: renamed from C1; value 0.1µF -> 100nF
- moved J3 205.7 mm to (362.6, -5.71), turned to 90 degrees
- moved J4 158.9 mm to (-13.8, -26.8)
- moved J2 14.7 mm to (371.2, 2.54), turned to 270 degrees
- renumbered C6 to C1, C7 to C2, C8 to C3, C9 to C4, C5 to C6, C4 to C7, C3 to C8, C2 to C9, IC6 to IC1, IC7 to IC2, IC8 to IC3, IC9 to IC4, IC1 to IC5, IC5 to IC6, IC4 to IC7, IC3 to IC8, IC2 to IC9, J3 to J1, J4 to J2, J2 to J3, J1 to J4, R6 to R1, R7 to R2, R8 to R3, R9 to R4, R4 to R6, R3 to R7, R2 to R8
Connections:
- J4 pad 3: SER -> QH
- J4 pad 4: QH -> SER

Commit message: Update PCB
Parts:
- J1: footprint Connector_PinHeader_2.54mm:PinHeader_1x04_P2.54mm_Horizontal -> Connector_PinSocket_2.54mm:PinSocket_1x04_P2.54mm_Horizontal; moved to B.Cu
- J2: moved to B.Cu
- J3: value Conn_01x06 -> Conn_01x05; footprint Connector_PinHeader_2.54mm:PinHeader_1x06_P2.54mm_Horizontal -> Connector_PinSocket_2.54mm:PinSocket_1x05_P2.54mm_Horizontal; moved to B.Cu
- J4: value Conn_01x06 -> Conn_01x05; footprint Connector_PinHeader_2.54mm:PinHeader_1x06_P2.54mm_Horizontal -> Connector_PinHeader_2.54mm:PinHeader_1x05_P2.54mm_Horizontal; moved to B.Cu
- moved J2 275.0 mm to (96.3, 8.00)
- moved J3 208.1 mm to (154.6, -9.02), turned to 270 degrees
- moved J4 172.0 mm to (154.6, 8.00), turned to 270 degrees
- moved J1 105.3 mm to (96.3, -9.02), turned to 270 degrees
- moved JP1 5.68 mm to (151.4, -9.74)
- moved IC5 4.09 mm to (161.9, 0.00)
- moved C5 2.91 mm to (157.0, -4.21), turned to 90 degrees
- moved R1 0.29 mm to (197.1, -4.56)
- moved C1 0.28 mm to (202.7, -4.57)
- moved C6 0.28 mm to (152.9, -4.57)
- moved C7 0.28 mm to (102.9, -4.57)
- moved C8 0.28 mm to (52.8, -4.57)
- moved C9 0.28 mm to (2.79, -4.57)
- moved R3 0.27 mm to (297.2, -4.57)
- moved R6 0.27 mm to (97.3, -4.57)
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Connections:
- J2 pad 1: Net-(D8-Pad6) -> GNDD
- J2 pad 2: Net-(D8-Pad5) -> +5V
- J2 pad 3: +5V -> Net-(D8-Pad5)
- J2 pad 4: GNDD -> Net-(D8-Pad6)
- J3 pad 3: QH -> SER
- J3 pad 4: SER -> CLK
- J3 pad 5: CLK -> SH
- J4 pad 1: SH -> GNDD
- J4 pad 2: CLK -> +3V3
- J4 pad 4: SER -> CLK
- J4 pad 5: +3V3 -> SH
Routing:
- net Net-(D8-Pad5): track 6.82 -> 260.1 mm
- net Net-(D8-Pad6): track 7.17 -> 260.3 mm
- net Net-(D1-Pad2): track 6.82 -> 127.2 mm
- net Net-(D1-Pad1): track 7.17 -> 116.3 mm
- net CLK: track 0.00 -> 30.4 mm
- net SER: track 0.00 -> 23.2 mm
- net +5V: track 382.5 -> 402.3 mm, vias 7 -> 16
- net SH: track 0.00 -> 19.1 mm
- net +3V3: track 379.3 -> 393.0 mm, vias 1 -> 2
- net GNDD: track 470.5 -> 481.4 mm, vias 1 -> 5
- net QH: track 0.00 -> 3.73 mm
- net Net-(IC1-Pad3): track 34.1 -> 35.9 mm
- net Net-(IC4-Pad3): track 185.9 -> 187.5 mm
- net Net-(IC2-Pad3): track 84.7 -> 86.4 mm
- net Net-(IC3-Pad3): track 135.4 -> 137.0 mm
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
Commit message: Schematic Update
Parts:
- J1: footprint Connector_PinSocket_2.54mm:PinSocket_1x04_P2.54mm_Horizontal -> Connector_PinHeader_2.54mm:PinHeader_1x04_P2.54mm_Horizontal; moved to F.Cu
- J2: footprint Connector_PinHeader_2.54mm:PinHeader_1x04_P2.54mm_Horizontal -> Connector_PinSocket_2.54mm:PinSocket_1x04_P2.54mm_Horizontal; moved to F.Cu
- J3: footprint Connector_PinSocket_2.54mm:PinSocket_1x05_P2.54mm_Horizontal -> Connector_PinHeader_2.54mm:PinHeader_1x05_P2.54mm_Horizontal; moved to F.Cu
- J4: footprint Connector_PinHeader_2.54mm:PinHeader_1x05_P2.54mm_Horizontal -> Connector_PinSocket_2.54mm:PinSocket_1x05_P2.54mm_Horizontal; moved to F.Cu
- moved J4 11.3 mm to (145.3, 14.5), turned to 90 degrees
- moved JP1 11.0 mm to (141.8, -15.0)
- moved J3 10.7 mm to (145.3, -14.4), turned to 90 degrees
- moved J2 6.54 mm to (96.2, 14.5), turned to 90 degrees
- moved R6 5.44 mm to (101.9, -7.49), turned to 180 degrees
- moved J1 5.33 mm to (96.3, -14.4), turned to 90 degrees
- moved C2 0.25 mm to (252.7, -4.59)
Routing:
- net CLK: track 30.4 -> 58.7 mm
- net GNDD: track 481.4 -> 509.4 mm
- net SH: track 19.1 -> 37.5 mm
- net +5V: track 402.3 -> 417.7 mm, vias 16 -> 15
- net +3V3: track 393.0 -> 406.9 mm
- net QH: track 3.73 -> 13.9 mm
- net SER: track 23.2 -> 33.0 mm
- net Net-(D1-Pad2): track 127.2 -> 118.5 mm
- net Net-(D8-Pad6): track 260.3 -> 265.8 mm
- net Net-(D8-Pad5): track 260.1 -> 264.6 mm
- net Net-(D1-Pad1): track 116.3 -> 117.2 mm
Other:
- board outline added: 400.3 x 50 mm

Commit message: Ontwerp Update
Parts:
- J1, J2, J3, J4: moved to B.Cu
- moved C1 175.5 mm to (27.2, -4.57)
- moved C5 175.5 mm to (-18.5, -4.21)
- moved C7 175.5 mm to (-72.6, -4.57)
- moved C8 175.5 mm to (-122.6, -4.57)
- moved C9 175.5 mm to (-172.7, -4.57)
- moved D1 175.5 mm to (-175.5, 0.00)
- moved D4 175.5 mm to (-25.3, 0.00)
- moved D5 175.5 mm to (24.4, 0.00)
- moved D6 175.5 mm to (74.5, 0.00)
- moved D8 175.5 mm to (174.6, 0.00)
- moved IC1 175.5 mm to (24.4, -4.56)
- moved IC2 175.5 mm to (74.5, -4.56)
- moved IC4 175.5 mm to (174.6, -4.56)
- moved IC5 175.5 mm to (-13.5, 0.00)
- moved IC6 175.5 mm to (-25.3, -4.56)
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Connections:
- J1 pad 1: GNDD -> Net-(D1-Pad1)
- J1 pad 2: +5V -> Net-(D1-Pad2)
- J1 pad 3: Net-(D1-Pad2) -> +5V
- J1 pad 4: Net-(D1-Pad1) -> GNDD
- J2 pad 1: GNDD -> Net-(D8-Pad6)
- J2 pad 2: +5V -> Net-(D8-Pad5)
- J2 pad 3: Net-(D8-Pad5) -> +5V
- J2 pad 4: Net-(D8-Pad6) -> GNDD
- J3 pad 1: GNDD -> SH
- J3 pad 2: +3V3 -> CLK
- J3 pad 4: CLK -> +3V3
- J3 pad 5: SH -> GNDD
- J4 pad 1: GNDD -> SH
- J4 pad 2: +3V3 -> CLK
- J4 pad 4: CLK -> +3V3
- J4 pad 5: SH -> GNDD
Routing:
- net GNDD: track 509.4 -> 512.1 mm
- added copper zone on B.Cu, net GNDD
- added copper zone on F.Cu, net GNDD
Other:
- board text added: "Schaakbord M.H."
