File: Schaakbord/Bord/Schaakbord_Bord.sch (KiCad schematic (older format))
At the start: 38 parts, among them IC1 SN74HC165DR, IC2 AH3572-SA-7, IC3 AH3572-SA-7, IC4 AH3572-SA-7, IC5 AH3572-SA-7, IC6 AH3572-SA-7, IC7 AH3572-SA-7, IC8 AH3572-SA-7, IC9 AH3572-SA-7, J1 Conn_01x06, J2 Conn_01x06, J3 Conn_01x04, J4 Conn_01x04

Commit message: Schematic Update
Parts:
- C1, C2, C3, C4, C5, C6, C7, C8, C9: footprint Capacitor_SMD:C_1206_3216Metric_Pad1.33x1.80mm_HandSolder -> Capacitor_SMD:C_0805_2012Metric_Pad1.18x1.45mm_HandSolder
- IC1: footprint Package_SO:SOP-16_3.9x9.9mm_P1.27mm -> SamacSys_Parts:SOIC127P600X175-16N
- R2, R3, R4, R5, R6, R7, R8, R9: footprint Resistor_SMD:R_1206_3216Metric_Pad1.30x1.75mm_HandSolder -> Resistor_SMD:R_0805_2012Metric_Pad1.20x1.40mm_HandSolder
Changed lines of the file:
@@
 F 0 "R5" H 9000 5250 50  0000 L CNN
 F 1 "10k" H 9000 5150 50  0000 L CNN
-F 2 "Resistor_SMD:R_1206_3216Metric_Pad1.30x1.75mm_HandSolder" V 8880 5200 50  0001 C CNN
+F 2 "Resistor_SMD:R_0805_2012Metric_Pad1.20x1.40mm_HandSolder" V 8880 5200 50  0001 C CNN
 F 3 "~" H 8950 5200 50  0001 C CNN
 	1    8950 5200
@@
 F 0 "R4" H 9000 5800 50  0000 L CNN
 F 1 "10k" H 9000 5700 50  0000 L CNN
-F 2 "Resistor_SMD:R_1206_3216Metric_Pad1.30x1.75mm_HandSolder" V 8880 5750 50  0001 C CNN
+F 2 "Resistor_SMD:R_0805_2012Metric_Pad1.20x1.40mm_HandSolder" V 8880 5750 50  0001 C CNN
 F 3 "~" H 8950 5750 50  0001 C CNN
 	1    8950 5750
@@
 F 0 "R3" H 9000 6350 50  0000 L CNN
 F 1 "10k" H 9000 6250 50  0000 L CNN
-F 2 "Resistor_SMD:R_1206_3216Metric_Pad1.30x1.75mm_HandSolder" V 8880 6300 50  0001 C CNN
+F 2 "Resistor_SMD:R_0805_2012Metric_Pad1.20x1.40mm_HandSolder" V 8880 6300 50  0001 C CNN
 F 3 "~" H 8950 6300 50  0001 C CNN
 	1    8950 6300
@@
 F 0 "R2" H 9000 6900 50  0000 L CNN
 F 1 "10k" H 9000 6800 50  0000 L CNN
-F 2 "Resistor_SMD:R_1206_3216Metric_Pad1.30x1.75mm_HandSolder" V 8880 6850 50  0001 C CNN
+F 2 "Resistor_SMD:R_0805_2012Metric_Pad1.20x1.40mm_HandSolder" V 8880 6850 50  0001 C CNN
 F 3 "~" H 8950 6850 50  0001 C CNN
 	1    8950 6850
@@
 F 0 "R6" H 6250 5250 50  0000 L CNN
 F 1 "10k" H 6250 5150 50  0000 L CNN
-F 2 "Resistor_SMD:R_1206_3216Metric_Pad1.30x1.75mm_HandSolder" V 6130 5200 50  0001 C CNN
+F 2 "Resistor_SMD:R_0805_2012Metric_Pad1.20x1.40mm_HandSolder" V 6130 5200 50  0001 C CNN
 F 3 "~" H 6200 5200 50  0001 C CNN
 	1    6200 5200
@@
 F 0 "R7" H 6250 5800 50  0000 L CNN
 F 1 "10k" H 6250 5700 50  0000 L CNN
-F 2 "Resistor_SMD:R_1206_3216Metric_Pad1.30x1.75mm_HandSolder" V 6130 5750 50  0001 C CNN
+F 2 "Resistor_SMD:R_0805_2012Metric_Pad1.20x1.40mm_HandSolder" V 6130 5750 50  0001 C CNN
 F 3 "~" H 6200 5750 50  0001 C CNN
 	1    6200 5750
@@
 F 0 "R8" H 6250 6350 50  0000 L CNN
 F 1 "10k" H 6250 6250 50  0000 L CNN
-F 2 "Resistor_SMD:R_1206_3216Metric_Pad1.30x1.75mm_HandSolder" V 6130 6300 50  0001 C CNN
+F 2 "Resistor_SMD:R_0805_2012Metric_Pad1.20x1.40mm_HandSolder" V 6130 6300 50  0001 C CNN
 F 3 "~" H 6200 6300 50  0001 C CNN
 	1    6200 6300
@@
 F 0 "R9" H 6250 6900 50  0000 L CNN
 F 1 "10k" H 6250 6800 50  0000 L CNN
-F 2 "Resistor_SMD:R_1206_3216Metric_Pad1.30x1.75mm_HandSolder" V 6130 6850 50  0001 C CNN
+F 2 "Resistor_SMD:R_0805_2012Metric_Pad1.20x1.40mm_HandSolder" V 6130 6850 50  0001 C CNN
 F 3 "~" H 6200 6850 50  0001 C CNN
 	1    6200 6850
@@
 F 0 "C1" H 8258 5604 50  0000 R CNN
 F 1 "0.1µF" H 8300 5700 50  0000 R CNN
-F 2 "Capacitor_SMD:C_1206_3216Metric_Pad1.33x1.80mm_HandSolder" H 8350 5650 50  0001 C CNN
+F 2 "Capacitor_SMD:C_0805_2012Metric_Pad1.18x1.45mm_HandSolder" H 8350 5650 50  0001 C CNN
 F 3 "~" H 8350 5650 50  0001 C CNN
 	1    8350 5650
@@
 Wire Wire Line
 	6800 5950 6550 5950
-$Comp
-L SamacSys_Parts:SN74HC165DR IC1
-U 1 1 603CFBAD
-P 6800 5750
-F 0 "IC1" H 7500 6015 50  0000 C CNN
-F 1 "SN74HC165DR" H 7500 5924 50  0000 C CNN
-F 2 "Package_SO:SOP-16_3.9x9.9mm_P1.27mm" H 8050 5850 50  0001 L CNN
-F 3 "http://www.ti.com/lit/ds/symlink/sn74hc165.pdf" H 8050 5750 50  0001 L CNN
-F 4 "8-Bit Parallel-Load Shift Registers" H 8050 5650 50  0001 L CNN "Description"
-F 5 "1.75" H 8050 5550 50  0001 L CNN "Height"
-F 6 "595-SN74HC165DR" H 8050 5450 50  0001 L CNN "Mouser Part Number"
-F 7 "https://www.mouser.co.uk/ProductDetail/Texas-Instruments/SN74HC165DR?qs=vxEfx8VrU7AaZtng63yj8Q%3D%3D" H 8050 5350 50  0001 L CNN "Mouser Price/Stock"
-F 8 "Texas Instruments" H 8050 5250 50  0001 L CNN "Manufacturer_Name"
-F 9 "SN74HC165DR" H 8050 5150 50  0001 L CNN "Manufacturer_Part_Number"
-	1    6800 5750
-	1    0    0    -1
-$EndComp
 $Comp
 L Device:C_Small C9
@@
 F 0 "C9" H 4900 7000 50  0000 R CNN
 F 1 "100nF" H 5050 7100 50  0000 R CNN
-F 2 "Capacitor_SMD:C_1206_3216Metric_Pad1.33x1.80mm_HandSolder" H 4700 7050 50  0001 C CNN
+F 2 "Capacitor_SMD:C_0805_2012Metric_Pad1.18x1.45mm_HandSolder" H 4700 7050 50  0001 C CNN
 F 3 "~" H 4700 7050 50  0001 C CNN
 	1    4700 7050
@@
 F 0 "C8" H 4900 6450 50  0000 R CNN
 F 1 "100nF" H 5050 6550 50  0000 R CNN
-F 2 "Capacitor_SMD:C_1206_3216Metric_Pad1.33x1.80mm_HandSolder" H 4700 6500 50  0001 C CNN
+F 2 "Capacitor_SMD:C_0805_2012Metric_Pad1.18x1.45mm_HandSolder" H 4700 6500 50  0001 C CNN
 F 3 "~" H 4700 6500 50  0001 C CNN
 	1    4700 6500
@@
 F 0 "C7" H 4900 5900 50  0000 R CNN
 F 1 "100nF" H 5050 6000 50  0000 R CNN
-F 2 "Capacitor_SMD:C_1206_3216Metric_Pad1.33x1.80mm_HandSolder" H 4700 5950 50  0001 C CNN
+F 2 "Capacitor_SMD:C_0805_2012Metric_Pad1.18x1.45mm_HandSolder" H 4700 5950 50  0001 C CNN
 F 3 "~" H 4700 5950 50  0001 C CNN
 	1    4700 5950
@@
 F 0 "C6" H 4900 5350 50  0000 R CNN
 F 1 "100nF" H 5050 5450 50  0000 R CNN
-F 2 "Capacitor_SMD:C_1206_3216Metric_Pad1.33x1.80mm_HandSolder" H 4700 5400 50  0001 C CNN
+F 2 "Capacitor_SMD:C_0805_2012Metric_Pad1.18x1.45mm_HandSolder" H 4700 5400 50  0001 C CNN
 F 3 "~" H 4700 5400 50  0001 C CNN
 	1    4700 5400
@@
 F 0 "C2" H 10650 7000 50  0000 R CNN
 F 1 "100nF" H 10800 7100 50  0000 R CNN
-F 2 "Capacitor_SMD:C_1206_3216Metric_Pad1.33x1.80mm_HandSolder" H 10450 7050 50  0001 C CNN
+F 2 "Capacitor_SMD:C_0805_2012Metric_Pad1.18x1.45mm_HandSolder" H 10450 7050 50  0001 C CNN
 F 3 "~" H 10450 7050 50  0001 C CNN
 	1    10450 7050
@@
 F 0 "C3" H 10650 6450 50  0000 R CNN
 F 1 "100nF" H 10800 6550 50  0000 R CNN
-F 2 "Capacitor_SMD:C_1206_3216Metric_Pad1.33x1.80mm_HandSolder" H 10450 6500 50  0001 C CNN
+F 2 "Capacitor_SMD:C_0805_2012Metric_Pad1.18x1.45mm_HandSolder" H 10450 6500 50  0001 C CNN
 F 3 "~" H 10450 6500 50  0001 C CNN
 	1    10450 6500
@@
 F 0 "C4" H 10650 5900 50  0000 R CNN
 F 1 "100nF" H 10800 6000 50  0000 R CNN
-F 2 "Capacitor_SMD:C_1206_3216Metric_Pad1.33x1.80mm_HandSolder" H 10450 5950 50  0001 C CNN
+F 2 "Capacitor_SMD:C_0805_2012Metric_Pad1.18x1.45mm_HandSolder" H 10450 5950 50  0001 C CNN
 F 3 "~" H 10450 5950 50  0001 C CNN
 	1    10450 5950
@@
 F 0 "C5" H 10650 5350 50  0000 R CNN
 F 1 "100nF" H 10800 5450 50  0000 R CNN
-F 2 "Capacitor_SMD:C_1206_3216Metric_Pad1.33x1.80mm_HandSolder" H 10450 5400 50  0001 C CNN
+F 2 "Capacitor_SMD:C_0805_2012Metric_Pad1.18x1.45mm_HandSolder" H 10450 5400 50  0001 C CNN
 F 3 "~" H 10450 5400 50  0001 C CNN
 	1    10450 5400
@@
 Wire Wire Line
 	8350 5750 8400 5750
+$Comp
+L SamacSys_Parts:SN74HC165DR IC1
+U 1 1 608BC4DC
+P 6800 5750
+F 0 "IC1" H 7500 6015 50  0000 C CNN
+F 1 "SN74HC165DR" H 7500 5924 50  0000 C CNN
+F 2 "SamacSys_Parts:SOIC127P600X175-16N" H 8050 5850 50  0001 L CNN
+F 3 "http://www.ti.com/lit/ds/symlink/sn74hc165.pdf" H 8050 5750 50  0001 L CNN
+F 4 "8-Bit Parallel-Load Shift Registers" H 8050 5650 50  0001 L CNN "Description"
+F 5 "1.75" H 8050 5550 50  0001 L CNN "Height"
+F 6 "595-SN74HC165DR" H 8050 5450 50  0001 L CNN "Mouser Part Number"
+F 7 "https://www.mouser.co.uk/ProductDetail/Texas-Instruments/SN74HC165DR?qs=vxEfx8VrU7AaZtng63yj8Q%3D%3D" H 8050 5350 50  0001 L CNN "Mouser Price/Stock"
+F 8 "Texas Instruments" H 8050 5250 50  0001 L CNN "Manufacturer_Name"
+F 9 "SN74HC165DR" H 8050 5150 50  0001 L CNN "Manufacturer_Part_Number"
+	1    6800 5750
+	1    0    0    -1
+$EndComp
 $EndSCHEMATC

Commit message: PCB
Parts:
- added JP1: Jumper, Jumper:SolderJumper-2_P1.3mm_Open_TrianglePad1.0x1.5mm, symbol Device:Jumper
- C5: renamed from C1; value 0.1µF -> 100nF
- renumbered C6 to C1, C7 to C2, C8 to C3, C9 to C4, C5 to C6, C4 to C7, C3 to C8, C2 to C9, IC6 to IC1, IC7 to IC2, IC8 to IC3, IC9 to IC4, IC1 to IC5, IC5 to IC6, IC4 to IC7, IC3 to IC8, IC2 to IC9, J3 to J1, J4 to J2, J2 to J3, J1 to J4, R6 to R1, R7 to R2, R8 to R3, R9 to R4, R4 to R6, R3 to R7, R2 to R8
Connections:
- net GNDD: now also JP1.2
- net QH: now also J4.3 (Pin_3); no longer J4.4 (Pin_4)
- net SER: now also J4.4 (Pin_4), JP1.1; no longer J4.3 (Pin_3)
Other:
- moved on the sheet: C5, R1, R2, R3, R4, R5, R6, R7, R8

Commit message: Update PCB
Parts:
- removed J3, J4: Conn_01x06, Connector_PinHeader_2.54mm:PinHeader_1x06_P2.54mm_Horizontal, symbol Connector_Generic:Conn_01x06
- added J3: Conn_01x05, Connector_PinSocket_2.54mm:PinSocket_1x05_P2.54mm_Horizontal, symbol Connector_Generic:Conn_01x05
- added J4: Conn_01x05, Connector_PinHeader_2.54mm:PinHeader_1x05_P2.54mm_Horizontal, symbol Connector_Generic:Conn_01x05
- J1: footprint Connector_PinHeader_2.54mm:PinHeader_1x04_P2.54mm_Horizontal -> Connector_PinSocket_2.54mm:PinSocket_1x04_P2.54mm_Horizontal
Connections:
- net +3V3: now also J3.2 (Pin_2), J4.2 (Pin_2)
- net +5V: now also J2.2 (Pin_2); no longer J2.3 (Pin_3)
- net CLK: now also J3.4 (Pin_4), J4.4 (Pin_4)
- net GNDD: now also J2.1 (Pin_1), J3.1 (Pin_1), J4.1 (Pin_1); no longer J2.4 (Pin_4)
- net QH: now also J4.3 (Pin_3)
- net SER: now also J3.3 (Pin_3)
- net SH: now also J3.5 (Pin_5), J4.5 (Pin_5)
- net at D8.5 (CO): now also J2.3 (Pin_3); no longer J2.2 (Pin_2)
- net at D8.6 (DO): now also J2.4 (Pin_4); no longer J2.1 (Pin_1)
Changed lines of the file:
@@
 L Connector_Generic:Conn_01x04 J2
 U 1 1 6087E1CF
-P 10950 3850
-F 0 "J2" H 11030 3842 50  0000 L CNN
-F 1 "Conn_01x04" H 11030 3751 50  0000 L CNN
-F 2 "Connector_PinHeader_2.54mm:PinHeader_1x04_P2.54mm_Horizontal" H 10950 3850 50  0001 C CNN
-F 3 "~" H 10950 3850 50  0001 C CNN
-	1    10950 3850
-	1    0    0    -1
+P 10950 3950
+F 0 "J2" H 11030 3942 50  0000 L CNN
+F 1 "Conn_01x04" H 11030 3851 50  0000 L CNN
+F 2 "Connector_PinHeader_2.54mm:PinHeader_1x04_P2.54mm_Horizontal" H 10950 3950 50  0001 C CNN
+F 3 "~" H 10950 3950 50  0001 C CNN
+	1    10950 3950
+	1    0    0    1
 $EndComp
 $Comp
@@
 F 0 "J1" H 5230 3942 50  0000 L CNN
 F 1 "Conn_01x04" H 5230 3851 50  0000 L CNN
-F 2 "Connector_PinHeader_2.54mm:PinHeader_1x04_P2.54mm_Horizontal" H 5150 3950 50  0001 C CNN
+F 2 "Connector_PinSocket_2.54mm:PinSocket_1x04_P2.54mm_Horizontal" H 5150 3950 50  0001 C CNN
 F 3 "~" H 5150 3950 50  0001 C CNN
 	1    5150 3950
@@
 Wire Wire Line
 	10700 3950 10750 3950
-$Comp
-L Connector_Generic:Conn_01x06 J4
-U 1 1 609D20CA
-P 11550 6500
-F 0 "J4" H 11630 6492 50  0000 L CNN
-F 1 "Conn_01x06" H 11630 6401 50  0000 L CNN
-F 2 "Connector_PinHeader_2.54mm:PinHeader_1x06_P2.54mm_Horizontal" H 11550 6500 50  0001 C CNN
-F 3 "~" H 11550 6500 50  0001 C CNN
-	1    11550 6500
-	1    0    0    -1
-$EndComp
 Text GLabel 11350 6300 0    50   Input ~ 0
 SH
 Text GLabel 11350 6400 0    50   Input ~ 0
 CLK
-Text GLabel 11350 6600 0    50   Input ~ 0
-SER
-Text GLabel 11350 6500 0    50   Input ~ 0
-QH
-$Comp
-L Connector_Generic:Conn_01x06 J3
-U 1 1 6072BFBE
-P 11550 5800
-F 0 "J3" H 11625 5675 50  0000 L CNN
-F 1 "Conn_01x06" H 11625 5750 50  0000 L CNN
-F 2 "Connector_PinHeader_2.54mm:PinHeader_1x06_P2.54mm_Horizontal" H 11550 5800 50  0001 C CNN
-F 3 "~" H 11550 5800 50  0001 C CNN
-	1    11550 5800
-	1    0    0    1
-$EndComp
-$Comp
-L power:+3V3 #PWR049
-U 1 1 609D20D0
-P 11050 6750
-F 0 "#PWR049" H 11050 6600 50  0001 C CNN
-F 1 "+3V3" H 11050 6900 50  0000 C CNN
-F 2 "" H 11050 6750 50  0001 C CNN
-F 3 "" H 11050 6750 50  0001 C CNN
-	1    11050 6750
-	-1   0    0    -1
-$EndComp
-Wire Wire Line
-	11050 6750 11200 6750
-Wire Wire Line
-	11200 6700 11350 6700
-Wire Wire Line
-	11200 6750 11200 6700
-$Comp
-L power:GNDD #PWR052
+$Comp
+L power:GNDD #PWR051
 U 1 1 609D20D6
-P 11350 6800
-F 0 "#PWR052" H 11350 6550 50  0001 C CNN
-F 1 "GNDD" H 11354 6645 50  0000 C CNN
-F 2 "" H 11350 6800 50  0001 C CNN
-F 3 "" H 11350 6800 50  0001 C CNN
-	1    11350 6800
+P 11350 6700
+F 0 "#PWR051" H 11350 6450 50  0001 C CNN
+F 1 "GNDD" H 11354 6545 50  0000 C CNN
+F 2 "" H 11350 6700 50  0001 C CNN
+F 3 "" H 11350 6700 50  0001 C CNN
+	1    11350 6700
 	-1   0    0    -1
 $EndComp
@@
 Text GLabel 11350 5700 0    50   Input ~ 0
 SER
-Text GLabel 11350 5800 0    50   Input ~ 0
-QH
 $Comp
 L power:+3V3 #PWR048
 U 1 1 60A12156
-P 11050 5950
-F 0 "#PWR048" H 11050 5800 50  0001 C CNN
-F 1 "+3V3" H 11050 6100 50  0000 C CNN
-F 2 "" H 11050 5950 50  0001 C CNN
-F 3 "" H 11050 5950 50  0001 C CNN
-	1    11050 5950
+P 11050 5850
+F 0 "#PWR048" H 11050 5700 50  0001 C CNN
+F 1 "+3V3" H 11050 6000 50  0000 C CNN
+F 2 "" H 11050 5850 50  0001 C CNN
+F 3 "" H 11050 5850 50  0001 C CNN
+	1    11050 5850
 	-1   0    0    -1
 $EndComp
 Wire Wire Line
-	11050 5950 11200 5950
-Wire Wire Line
-	11200 5900 11350 5900
-Wire Wire Line
-	11200 5950 11200 5900
-$Comp
-L power:GNDD #PWR051
+	11050 5850 11200 5850
+Wire Wire Line
+	11200 5800 11350 5800
+Wire Wire Line
+	11200 5850 11200 5800
+$Comp
+L power:GNDD #PWR050
 U 1 1 60A1215F
-P 11350 6000
-F 0 "#PWR051" H 11350 5750 50  0001 C CNN
-F 1 "GNDD" H 11354 5845 50  0000 C CNN
-F 2 "" H 11350 6000 50  0001 C CNN
-F 3 "" H 11350 6000 50  0001 C CNN
-	1    11350 6000
+P 11350 5900
+F 0 "#PWR050" H 11350 5650 50  0001 C CNN
+F 1 "GNDD" H 11354 5745 50  0000 C CNN
+F 2 "" H 11350 5900 50  0001 C CNN
+F 3 "" H 11350 5900 50  0001 C CNN
+	1    11350 5900
 	-1   0    0    -1
 $EndComp
@@
 SER
 $Comp
-L power:GNDD #PWR050
+L power:GNDD #PWR052
 U 1 1 609D449A
 P 11800 5175
-F 0 "#PWR050" H 11800 4925 50  0001 C CNN
+F 0 "#PWR052" H 11800 4925 50  0001 C CNN
 F 1 "GNDD" H 11804 5020 50  0000 C CNN
 F 2 "" H 11800 5175 50  0001 C CNN
@@
 	1    0    0    -1
 $EndComp
+Text GLabel 11350 6500 0    50   Input ~ 0
+QH
+$Comp
+L Connector_Generic:Conn_01x05 J4
+U 1 1 60A52C76
+P 11550 6500
+F 0 "J4" H 11468 6075 50  0000 C CNN
+F 1 "Conn_01x05" H 11468 6166 50  0000 C CNN
+F 2 "Connector_PinHeader_2.54mm:PinHeader_1x05_P2.54mm_Horizontal" H 11550 6500 50  0001 C CNN
+F 3 "~" H 11550 6500 50  0001 C CNN
+	1    11550 6500
+	1    0    0    1
+$EndComp
+$Comp
+L Connector_Generic:Conn_01x05 J3
+U 1 1 60A596AF
+P 11550 5700
+F 0 "J3" H 11468 5275 50  0000 C CNN
+F 1 "Conn_01x05" H 11468 5366 50  0000 C CNN
+F 2 "Connector_PinSocket_2.54mm:PinSocket_1x05_P2.54mm_Horizontal" H 11550 5700 50  0001 C CNN
+F 3 "~" H 11550 5700 50  0001 C CNN
+	1    11550 5700
+	1    0    0    1
+$EndComp
+$Comp
+L power:+3V3 #PWR049
+U 1 1 609D20D0
+P 11050 6650
+F 0 "#PWR049" H 11050 6500 50  0001 C CNN
+F 1 "+3V3" H 11050 6800 50  0000 C CNN
+F 2 "" H 11050 6650 50  0001 C CNN
+F 3 "" H 11050 6650 50  0001 C CNN
+	1    11050 6650
+	-1   0    0    -1
+$EndComp
+Wire Wire Line
+	11200 6600 11350 6600
+Wire Wire Line
+	11200 6650 11200 6600
+Wire Wire Line
+	11050 6650 11200 6650
 $EndSCHEMATC

Commit message: Schematic Update
Parts:
- J1: footprint Connector_PinSocket_2.54mm:PinSocket_1x04_P2.54mm_Horizontal -> Connector_PinHeader_2.54mm:PinHeader_1x04_P2.54mm_Horizontal
- J2: footprint Connector_PinHeader_2.54mm:PinHeader_1x04_P2.54mm_Horizontal -> Connector_PinSocket_2.54mm:PinSocket_1x04_P2.54mm_Horizontal
- J3: footprint Connector_PinSocket_2.54mm:PinSocket_1x05_P2.54mm_Horizontal -> Connector_PinHeader_2.54mm:PinHeader_1x05_P2.54mm_Horizontal
- J4: footprint Connector_PinHeader_2.54mm:PinHeader_1x05_P2.54mm_Horizontal -> Connector_PinSocket_2.54mm:PinSocket_1x05_P2.54mm_Horizontal
Changed lines of the file:
@@
 	10550 3750 10750 3750
-$Comp
-L Connector_Generic:Conn_01x04 J2
-U 1 1 6087E1CF
-P 10950 3950
-F 0 "J2" H 11030 3942 50  0000 L CNN
-F 1 "Conn_01x04" H 11030 3851 50  0000 L CNN
-F 2 "Connector_PinHeader_2.54mm:PinHeader_1x04_P2.54mm_Horizontal" H 10950 3950 50  0001 C CNN
-F 3 "~" H 10950 3950 50  0001 C CNN
-	1    10950 3950
-	1    0    0    1
-$EndComp
 $Comp
 L Device:C_Small C5
@@
 	1    5500 4050
 	1    0    0    -1
-$EndComp
-$Comp
-L Connector_Generic:Conn_01x04 J1
-U 1 1 6072E135
-P 5150 3950
-F 0 "J1" H 5230 3942 50  0000 L CNN
-F 1 "Conn_01x04" H 5230 3851 50  0000 L CNN
-F 2 "Connector_PinSocket_2.54mm:PinSocket_1x04_P2.54mm_Horizontal" H 5150 3950 50  0001 C CNN
-F 3 "~" H 5150 3950 50  0001 C CNN
-	1    5150 3950
-	-1   0    0    1
 $EndComp
 Wire Wire Line
@@
 QH
 $Comp
-L Connector_Generic:Conn_01x05 J4
-U 1 1 60A52C76
-P 11550 6500
-F 0 "J4" H 11468 6075 50  0000 C CNN
-F 1 "Conn_01x05" H 11468 6166 50  0000 C CNN
-F 2 "Connector_PinHeader_2.54mm:PinHeader_1x05_P2.54mm_Horizontal" H 11550 6500 50  0001 C CNN
-F 3 "~" H 11550 6500 50  0001 C CNN
-	1    11550 6500
-	1    0    0    1
-$EndComp
-$Comp
-L Connector_Generic:Conn_01x05 J3
-U 1 1 60A596AF
-P 11550 5700
-F 0 "J3" H 11468 5275 50  0000 C CNN
-F 1 "Conn_01x05" H 11468 5366 50  0000 C CNN
-F 2 "Connector_PinSocket_2.54mm:PinSocket_1x05_P2.54mm_Horizontal" H 11550 5700 50  0001 C CNN
-F 3 "~" H 11550 5700 50  0001 C CNN
-	1    11550 5700
-	1    0    0    1
-$EndComp
-$Comp
 L power:+3V3 #PWR049
 U 1 1 609D20D0
@@
 Wire Wire Line
 	11050 6650 11200 6650
+$Comp
+L Connector_Generic:Conn_01x04 J1
+U 1 1 6072E135
+P 5150 3950
+F 0 "J1" H 5230 3942 50  0000 L CNN
+F 1 "Conn_01x04" H 5230 3851 50  0000 L CNN
+F 2 "Connector_PinHeader_2.54mm:PinHeader_1x04_P2.54mm_Horizontal" H 5150 3950 50  0001 C CNN
+F 3 "~" H 5150 3950 50  0001 C CNN
+	1    5150 3950
+	-1   0    0    1
+$EndComp
+$Comp
+L Connector_Generic:Conn_01x04 J2
+U 1 1 6087E1CF
+P 10950 3950
+F 0 "J2" H 11030 3942 50  0000 L CNN
+F 1 "Conn_01x04" H 11030 3851 50  0000 L CNN
+F 2 "Connector_PinSocket_2.54mm:PinSocket_1x04_P2.54mm_Horizontal" H 10950 3950 50  0001 C CNN
+F 3 "~" H 10950 3950 50  0001 C CNN
+	1    10950 3950
+	1    0    0    1
+$EndComp
+$Comp
+L Connector_Generic:Conn_01x05 J3
+U 1 1 60A596AF
+P 11550 5700
+F 0 "J3" H 11468 5275 50  0000 C CNN
+F 1 "Conn_01x05" H 11468 5366 50  0000 C CNN
+F 2 "Connector_PinHeader_2.54mm:PinHeader_1x05_P2.54mm_Horizontal" H 11550 5700 50  0001 C CNN
+F 3 "~" H 11550 5700 50  0001 C CNN
+	1    11550 5700
+	1    0    0    1
+$EndComp
+$Comp
+L Connector_Generic:Conn_01x05 J4
+U 1 1 60A52C76
+P 11550 6500
+F 0 "J4" H 11468 6075 50  0000 C CNN
+F 1 "Conn_01x05" H 11468 6166 50  0000 C CNN
+F 2 "Connector_PinSocket_2.54mm:PinSocket_1x05_P2.54mm_Horizontal" H 11550 6500 50  0001 C CNN
+F 3 "~" H 11550 6500 50  0001 C CNN
+	1    11550 6500
+	1    0    0    1
+$EndComp
 $EndSCHEMATC
